File: hardware/tagbase-lipo-v1/tagbase-lipo-v1.kicad_pcb (KiCad board)
At the start: 2 copper layers, 50.8 x 69.9 mm, 38 parts, among them J1 Conn_01x04_Female, J101 Conn_02x03_Odd_Even, J102 Conn_02x05_Odd_Even, J104 USB_B_Mini, J2 Conn_01x06, J5 Conn_01x02, SW1 SW_SPDT, SW2 SW_SPDT, U1 XC6206P332MR, U105 Tactile Switch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

Commit message: update tagbase lipo design
Parts:
- removed C107: 0.1uF, Capacitor_SMD:C_0402_1005Metric
- removed C7: 4.7uf, Capacitor_SMD:C_0402_1005Metric
- added U5: SN74LVC1T45DCK, Package_TO_SOT_SMD:SOT-23-6, F.Cu at (119.1, 69.3)
- added U6: SN74LVC1T45DCK, Package_TO_SOT_SMD:SOT-23-6, F.Cu at (124.0, 69.3)
- R4: value 1K -> 100
- U3: value XC6206P202MR -> XC6206P182MR
- U4: value STM32C071GBU6N -> STM32C071GBUx
- moved C4 37.5 mm to (105.1, 69.3), turned to -90 degrees
- moved C1 35.9 mm to (105.1, 72.1), turned to 90 degrees
- moved U3 34.6 mm to (107.7, 68.7), turned to 180 degrees
- moved U1 32.2 mm to (107.7, 72.4), turned to 180 degrees
- moved C5 31.5 mm to (110.4, 68.7), turned to -90 degrees
- moved C104 28.8 mm to (110.4, 72.4), turned to 90 degrees
- moved J5 26.3 mm to (140.0, 63.0), turned to -90 degrees
- moved R3 15.7 mm to (132.5, 68.7), turned to 90 degrees
- moved R2 12.6 mm to (142.9, 67.2), turned to 0 degrees
- moved U2 11.6 mm to (140.2, 67.6)
- moved R1 11.0 mm to (142.9, 68.3), turned to 0 degrees
- moved D105 8.05 mm to (110.0, 76.7)
- moved R5 8.05 mm to (107.8, 76.8)
- moved SW1 7.86 mm to (136.4, 72.7), turned to 180 degrees
- moved R4 6.09 mm to (127.2, 64.9), turned to 180 degrees
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Connections:
- C2 pad 1: +2V -> +3V3
- C5 pad 1: +2V -> +1V8
- C6 pad 1: +2V -> +3V3
- R104 pad 2: Net-(U4-PB7) -> Net-(U4-PB8)
- R3 pad 1: +2V -> +3V3
- R4 pad 1: Net-(U4-PA2) -> Net-(U4-PB5)
- R4 pad 2: TAG_SWDIO -> Net-(U4-PB4)
- SW2 pad 1: /BAT -> unconnected-(SW2-A-Pad1)
- SW2 pad 3: unconnected-(SW2-C-Pad3) -> /BAT
- U3 pad 2: +2V -> +1V8
- U4 pad 10: TAG_SWDIO -> unconnected-(U4-PA4-Pad10)
- U4 pad 11: /CSO -> unconnected-(U4-PA5-Pad11)
- U4 pad 12: /CSO -> unconnected-(U4-PA6-Pad12)
- U4 pad 17: +3V3 -> unconnected-(U4-PC6-Pad17)
- U4 pad 23: unconnected-(U4-PB3-Pad23) -> Net-(U4-PB3)
- U4 pad 24: unconnected-(U4-PB4-Pad24) -> Net-(U4-PB4)
- U4 pad 25: unconnected-(U4-PB5-Pad25) -> Net-(U4-PB5)
- U4 pad 26: /UART_TX -> unconnected-(U4-PB6-Pad26)
- U4 pad 28: unconnected-(U4-PB8-Pad28) -> Net-(U4-PB8)
- U4 pad 3: +2V -> +3V3
- U4 pad 6: TAG_SCK -> /CSO
- U4 pad 7: TAG_SCK -> unconnected-(U4-PA1-Pad7)
- U4 pad 8: Net-(U4-PA2) -> /UART_TX
Routing:
- net +3V3: track 89.5 -> 231.2 mm, vias 2 -> 0
- net +2V: track 36.2 -> 0.00 mm, vias 4 -> 0
- net VUSB: track 35.7 -> 67.3 mm
- net +1V8: track 0.00 -> 24.6 mm, vias 0 -> 2
- net Net-(U4-PB3): track 0.00 -> 18.1 mm
- net /CSO: track 24.5 -> 8.57 mm, vias 2 -> 0
- net Net-(U4-PB4): track 0.00 -> 10.3 mm
- net TAG_SWDIO: track 45.3 -> 35.3 mm, vias 2 -> 1
- net TAG_3V3_IN: track 18.6 -> 23.2 mm, vias 1 -> 0
- net Net-(U4-PB7): track 1.62 -> 6.05 mm
- net /UART_TX: track 10.5 -> 6.11 mm, vias 1 -> 0
- net TAG_RESET: track 37.4 -> 33.4 mm, vias 3 -> 1
- net Net-(U4-PB8): track 0.00 -> 3.82 mm
- net /LED_GREEN: track 16.1 -> 12.3 mm
- net Net-(U4-PA2): track 3.71 -> 0.00 mm
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Other:
- board text added: "For Power Measurement: switch to pwr measure, no charge"
- board text added: "No Chg"
- board text removed: "NC"

Commit message: added torpor tag
Parts:
- R4: footprint Resistor_SMD:R_0402_1005Metric -> Resistor_SMD:R_0603_1608Metric
- U4: footprint tagbase:UFQFPN-28_STM -> Package_DFN_QFN:QFN-28_4x4mm_P0.5mm
- U5, U6: footprint Package_TO_SOT_SMD:SOT-23-6 -> Package_TO_SOT_SMD:SOT-363_SC-70-6
- moved R4 2.43 mm to (124.8, 65.3)
Routing:
- net +1V8: track 24.6 -> 19.4 mm, vias 2 -> 3
- net Net-(U4-PB5): track 1.36 -> 3.63 mm
- net Net-(U4-PB4): track 10.3 -> 10.8 mm
- net +3V3: track 231.2 -> 231.7 mm
