File: hardware/TorporTagBreakout/TorperTagBreakout.kicad_sch (KiCad schematic)
At the start: 16 parts, among them J3 Conn_01x17, J4 Conn_01x17, U1 AT25XE321D-UUN-T, U2 adxl362, U3 TMP119AIYBGR

Commit message: rearrange tag libraries
Parts:
- U2: footprint tag_ibrary:ADXL362 -> tag_library:ADXL362
Changed lines of the file:
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@@
 			)
 		)
-		(property "Footprint" "tag_ibrary:ADXL362"
+		(property "Footprint" "tag_library:ADXL362"
 			(at 64.77 125.73 0)
 			(hide yes)
