File: hardware/TorporTag/TorporTag.kicad_pcb (KiCad board)
At the start: 2 copper layers, 18 x 9 mm, 23 parts, among them J201 CONN_02X04, J301 Conn_01x01, J302 Conn_01x01, J303 Conn_01x01, J304 Conn_01x01, J401 CONN_01X02, Q501 Q_NPN_BEC, U1 at25ex321D-UUN, U2 adxl362, U3 TMP119AIYBGR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

Commit message: changed TorporTag to using local library
Parts:
- U1: footprint AccelTag:adesto_wlcsp12 -> tag_fp:adesto_wlcsp12

Commit message: rearrange tag libraries
Parts:
- D401: footprint Diode_SMD:D_0402_1005Metric -> tag_fp:D_0402_1005Metric
- Q501: footprint Package_TO_SOT_SMD:SOT-883 -> tag_fp:SOT-883
- U501: footprint AccelTag:RV-8803-C7 -> tag_fp:RV-8803-C7

Commit message: big checking after adding codex skills
Parts:
- removed C5: 0.1uf, Capacitor_SMD:C_0201_0603Metric
- J201: footprint AccelTag:tagpoints6 -> tag_fp:tagpoints6
- U2: footprint AccelTag:ADXL362 -> tag_fp:ADXL362
Connections:
- U2 pad 2: GND -> unconnected-(U2-NC-Pad2)
Routing:
- net GND: track 60.9 -> 55.0 mm
- added copper zone on B.Cu, net GND
- added copper zone on F.Cu, net VIN
Other:
- board text added: "TorporTag v1"
- board text removed: "TTag v1"
