File: hardware/TorporTag/TorporTag.kicad_sch (KiCad schematic)
At the start: 23 parts, among them J201 CONN_02X04, J301 Conn_01x01, J302 Conn_01x01, J303 Conn_01x01, J304 Conn_01x01, J401 CONN_01X02, Q501 Q_NPN_BEC, U1 at25ex321D-UUN, U2 adxl362, U3 TMP119AIYBGR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

Commit message: changed TorporTag to using local library
Parts:
- C5: DISTPN (none) -> 490-3167-1-ND; LCSC (none) -> C76928; MFN (none) -> Murata; MPN CL05F104ZO5NNNC -> GRM033R60J104KE19D
- J201: now in the parts list
- U1: footprint AccelTag:adesto_wlcsp12 -> tag_fp:adesto_wlcsp12; symbol BitTagNG:at25ex321D-UUN-AccelTag -> tag_library:at25ex321D-UUN
- U2: symbol bittagv7:adxl362 -> tag_library:adxl362; LCSC (none) -> C192252
- U3: LCSC (none) -> C22428347; MFN (none) -> Texas Instruments; MPN (none) -> TMP119AIYBGR
- U302: symbol BitTagNG:stm32l432-AccelTag -> tag_library:stm32l432
- U501: footprint AccelTag:RV-8803-C7 -> bittagv7:RV-8803-C7; symbol BitTagNG:RV-3028-C7-AccelTag -> tag_library:RV-3028-C7

Commit message: rearrange tag libraries
Parts:
- D401: footprint Diode_SMD:D_0402_1005Metric -> tag_fp:D_0402_1005Metric
- Q501: footprint Package_TO_SOT_SMD:SOT-883 -> tag_fp:SOT-883
- U501: footprint bittagv7:RV-8803-C7 -> tag_fp:RV-8803-C7
Changed lines of the file:
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@@
 			)
 		)
-		(property "Footprint" "Package_TO_SOT_SMD:SOT-883"
+		(property "Footprint" "tag_fp:SOT-883"
 			(at 49.53 90.17 0)
 			(hide yes)
@@
 			)
 		)
-		(property "Footprint" "Diode_SMD:D_0402_1005Metric"
+		(property "Footprint" "tag_fp:D_0402_1005Metric"
 			(at 231.14 33.02 0)
 			(hide yes)
@@
 			)
 		)
-		(property "Footprint" "bittagv7:RV-8803-C7"
+		(property "Footprint" "tag_fp:RV-8803-C7"
 			(at 218.44 127 0)
 			(hide yes)

Commit message: big checking after adding codex skills
Parts:
- removed C5: 0.1uf, Capacitor_SMD:C_0201_0603Metric, symbol Device:C
- J201: footprint AccelTag:tagpoints6 -> tag_fp:tagpoints6
- U2: footprint AccelTag:ADXL362 -> tag_fp:ADXL362
Connections:
- net GND: no longer U2.2 (NC)
- no-connect marks 12 -> 13
