File: hardware/CompassTag/CompassTag.kicad_pcb (KiCad board)
At the start: 2 copper layers, 18 x 9 mm, 28 parts, among them J201 CONN_02X04, J301 Conn_01x01, J302 Conn_01x01, J303 Conn_01x01, J304 Conn_01x01, J401 CONN_01X02, Q501 Q_NPN_BEC, U1 at25ex321D-UUN, U2 AK09940A, U3 LIS2DU12TR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

Commit message: update tagbase lipo design
Other:
- board text added: "CTag V2"
- board text removed: "CTag V1"

Commit message: Update CompassTag
Parts:
- U2: footprint AccelTag:AK09940a -> tag_fp:AK09940a
- U3: footprint AccelTag:LGA-12L_LIS2DU12_STM -> tag_fp:LGA-12L_LIS2DU12_STM
- U501: footprint AccelTag:RV-8803-C7 -> tag_fp:RV-8803-C7
Connections:
- net VIN renamed +2V5
Routing:
- net GND: track 60.0 -> 57.9 mm, vias 8 -> 9
- net /SCL: track 1.28 -> 1.81 mm
- added copper zone on F.Cu, net +2V5
- added copper zone on B.Cu, net GND
