File: hardware/CompassTag/CompassTag.kicad_sch (KiCad schematic)
At the start: 28 parts, among them J201 CONN_02X04, J301 Conn_01x01, J302 Conn_01x01, J303 Conn_01x01, J304 Conn_01x01, J401 CONN_01X02, Q501 Q_NPN_BEC, U1 at25ex321D-UUN, U2 AK09940A, U3 LIS2DU12TR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

Commit message: update tagbase lipo design
Parts:
- C1, C2, C3, C5, C501, C502, C503, C9: DISTPN 490-7229-1-ND -> 490-3167-1-ND; LCSC C181047 -> C76928; MPN GRM033R60J105MEA2D -> GRM033R60J104KE19D
- C6: LCSC (none) -> C140782; MFN KYOCERA AVX -> Murata; MPN 06036D476MAT2A -> GRM188R60J476ME15D
- C7, C8: LCSC (none) -> C126620
- Q501: DISTPN 1727-2632-1-ND -> 1727-PMBT2222AMBYLCT-ND; LCSC C686658 -> C552701; MPN BC847AMB,315 -> PMBT2222AMBYL
- U4: DISTPN 296-TPS7A2018PDQNRCT-ND -> 296-TPS7A0218PDQNRCT-ND; LCSC (none) -> C2862166; MPN TPS7A2018PDQNR -> TPS7A0218PDQNR
Changed lines of the file:
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@@
 			)
 		)
-		(property "MPN" "GRM033R60J105MEA2D"
+		(property "MPN" "GRM033R60J104KE19D"
 			(at 60.96 97.79 0)
 			(effects
@@
 			)
 		)
-		(property "DISTPN" "490-7229-1-ND"
+		(property "DISTPN" "490-3167-1-ND"
 			(at 0 195.58 0)
 			(effects
@@
 			)
 		)
-		(property "LCSC" "C181047"
+		(property "LCSC" "C76928"
 			(at 60.96 97.79 0)
 			(effects
@@
 			)
 		)
-		(property "MPN" "GRM033R60J105MEA2D"
+		(property "MPN" "GRM033R60J104KE19D"
 			(at 68.58 97.79 0)
 			(effects
@@
 			)
 		)
-		(property "DISTPN" "490-7229-1-ND"
+		(property "DISTPN" "490-3167-1-ND"
 			(at 0 195.58 0)
 			(effects
@@
 			)
 		)
-		(property "LCSC" "C181047"
+		(property "LCSC" "C76928"
 			(at 68.58 97.79 0)
 			(effects
@@
 			)
 		)
-		(property "MPN" "BC847AMB,315"
+		(property "MPN" "PMBT2222AMBYL"
 			(at 44.45 92.71 0)
 			(effects
@@
 			)
 		)
-		(property "DISTPN" "1727-2632-1-ND"
+		(property "DISTPN" "1727-PMBT2222AMBYLCT-ND"
 			(at 0 185.42 0)
 			(effects
@@
 			)
 		)
-		(property "LCSC" "C686658"
+		(property "LCSC" "C552701"
 			(at 44.45 92.71 0)
 			(effects
@@
 			)
 		)
-		(property "MPN" "GRM033R60J105MEA2D"
+		(property "MPN" "GRM033R60J104KE19D"
 			(at 256.54 134.62 0)
 			(effects
@@
 			)
 		)
-		(property "DISTPN" "490-7229-1-ND"
+		(property "DISTPN" "490-3167-1-ND"
 			(at 168.91 297.18 0)
 			(effects
@@
 			)
 		)
-		(property "LCSC" "C181047"
+		(property "LCSC" "C76928"
 			(at 256.54 134.62 0)
 			(effects
@@
 			)
 		)
-		(property "DISTPN" "490-7229-1-ND"
+		(property "DISTPN" "490-3167-1-ND"
 			(at 313.69 280.67 0)
 			(effects
@@
 			)
 		)
-		(property "MPN" "GRM033R60J105MEA2D"
+		(property "MPN" "GRM033R60J104KE19D"
 			(at 313.69 280.67 0)
 			(effects
@@
 			)
 		)
-		(property "LCSC" "C181047"
+		(property "LCSC" "C76928"
 			(at 135.89 177.8 0)
 			(effects
@@
 			)
 		)
-		(property "MPN" "GRM033R60J105MEA2D"
+		(property "MPN" "GRM033R60J104KE19D"
 			(at 165.1 101.6 0)
 			(effects
@@
 			)
 		)
-		(property "DISTPN" "490-7229-1-ND"
+		(property "DISTPN" "490-3167-1-ND"
 			(at 96.52 199.39 0)
 			(effects
@@
 			)
 		)
-		(property "LCSC" "C181047"
+		(property "LCSC" "C76928"
 			(at 165.1 101.6 0)
 			(effects
@@
 			)
 		)
-		(property "MPN" "GRM033R60J105MEA2D"
+		(property "MPN" "GRM033R60J104KE19D"
 			(at 257.81 86.36 0)
 			(effects
@@
 			)
 		)
-		(property "DISTPN" "490-7229-1-ND"
+		(property "DISTPN" "490-3167-1-ND"
 			(at 189.23 184.15 0)
 			(effects
@@
 			)
 		)
-		(property "LCSC" "C181047"
+		(property "LCSC" "C76928"
 			(at 257.81 86.36 0)
 			(effects
@@
 			)
 		)
-		(property "LCSC" ""
+		(property "LCSC" "C126620"
 			(at 251.46 86.36 0)
 			(effects
@@
 			)
 		)
-		(property "MPN" "GRM033R60J105MEA2D"
+		(property "MPN" "GRM033R60J104KE19D"
 			(at 101.6 132.08 0)
 			(effects
@@
 			)
 		)
-		(property "DISTPN" "490-7229-1-ND"
+		(property "DISTPN" "490-3167-1-ND"
 			(at 33.02 229.87 0)
 			(effects
@@
 			)
 		)
-		(property "LCSC" "C181047"
+		(property "LCSC" "C76928"
 			(at 101.6 132.08 0)
 			(effects
@@
 			)
 		)
-		(property "LCSC" ""
+		(property "LCSC" "C126620"
 			(at 218.44 86.36 0)
 			(effects
@@
 			)
 		)
-		(property "MFN" "KYOCERA AVX"
+		(property "MFN" "Murata"
 			(at 236.22 39.37 0)
 			(effects
@@
 			)
 		)
-		(property "MPN" "06036D476MAT2A"
+		(property "MPN" "GRM188R60J476ME15D"
 			(at 236.22 39.37 0)
 			(effects
@@
 			)
 		)
+		(property "LCSC" "C140782"
+			(at 236.22 39.37 0)
+			(effects
+				(font
+					(size 1.27 1.27)
+				)
+				(hide yes)
+			)
+		)
 		(pin "1"
 		)
@@
 			)
 		)
-		(property "MPN" "TPS7A2018PDQNR"
+		(property "MPN" "TPS7A0218PDQNR"
+			(at 240.03 83.82 0)
+			(effects
+				(font
+					(size 1.27 1.27)
+				)
+				(hide yes)
+			)
+		)
+		(property "DISTPN" "296-TPS7A0218PDQNRCT-ND"
 			(at 240.03 83.82 0)
 			(effects
@@
 			)
 		)
-		(property "DISTPN" "296-TPS7A2018PDQNRCT-ND"
+		(property "LCSC" "C2862166"
 			(at 240.03 83.82 0)
 			(effects
@@
 			)
 		)
-		(property "DISTPN" "490-7229-1-ND"
+		(property "DISTPN" "490-3167-1-ND"
 			(at 320.04 280.67 0)
 			(effects
@@
 			)
 		)
-		(property "MPN" "GRM033R60J105MEA2D"
+		(property "MPN" "GRM033R60J104KE19D"
 			(at 320.04 280.67 0)
 			(effects
@@
 			)
 		)
-		(property "LCSC" "C181047"
+		(property "LCSC" "C76928"
 			(at 142.24 177.8 0)
 			(effects

Commit message: Update CompassTag
Parts:
- Q501: symbol Device:Q_NPN_BEC -> Transistor_BJT:Q_NPN_BEC
- U1: symbol BitTagNG:at25ex321D-UUN-AccelTag -> tag_library:at25ex321D-UUN
- U2: footprint LGA11_1p6x1p6x0p58_AKM -> tag_fp:AK09940a; symbol ak09940a:AK09940A -> tag_library:AK09940A
- U3: footprint LGA-12L_LIS2DU12_STM -> tag_fp:LGA-12L_LIS2DU12_STM; symbol lis2du12:LIS2DU12TR -> tag_library:LIS2DU12TR
- U302: symbol BitTagNG:stm32l432-AccelTag -> tag_library:stm32l432
- U501: footprint AccelTag:RV-8803-C7 -> tag_fp:RV-8803-C7; symbol BitTagNG:RV-3028-C7-AccelTag -> tag_library:RV-3028-C7
Other:
- note added: "VIN=2V5"
