File: BoardDesigns/imutag/imutag.kicad_sch (KiCad schematic)
At the start: 27 parts, among them J201 CONN_02X04, J301 Conn_01x01, J302 Conn_01x01, J303 Conn_01x01, J304 Conn_01x01, J401 CONN_01X02, Q501 Q_NPN_BEC, U2 AK09940A, U3 LPS22DF, U302 stm32l431kc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

Commit message: new lipo breakout
Parts:
- U6: value ~ -> (none)
Other:
- note added: "Note, sda, scl intentionally swapped from hardware"
