File: BoardDesigns/IMUBreakout-v2/IMUBreakout-v2.kicad_pcb (KiCad board)
At the start: 4 copper layers, 48.3 x 48.3 mm, 15 parts, among them J3 Conn_01x17, J4 Conn_01x17, U2 MX25U12843GBBI00, U3 AK09940A, U4 LSM6DSV16XTR, U5 LPS22HH

Commit message: IMUBreakout and tag-breakout-l432-lipo-v1 submit for fab
Routing:
- net /LPS_CS: track 29.9 -> 23.9 mm, vias 0 -> 2
- net /MX_MISO: track 30.1 -> 25.3 mm, vias 0 -> 2
- net +1V8: track 24.1 -> 22.0 mm
- net GND: track 21.9 -> 20.9 mm, vias 19 -> 36
- net /MX_MOSI: track 23.0 -> 22.3 mm
- net /LSM_CK: track 44.4 -> 43.8 mm
