File: BoardDesigns/IMUBreakout-v2/IMUBreakout-v2.kicad_sch (KiCad schematic)
At the start: 15 parts, among them J3 Conn_01x17, J4 Conn_01x17, U2 MX25U12843GBBI00, U3 AK09940A, U4 LSM6DSV16XTR, U5 LPS22HH

Commit message: added new breakout board and imu tag with nand
Other:
- title: IMU Tag Breakout (3.3v) -> IMU Tag Breakout (1.8v)
Changed lines of the file:
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@@
 	(paper "A")
 	(title_block
-		(title "IMU Tag Breakout (3.3v)")
+		(title "IMU Tag Breakout (1.8v)")
 		(date "2026-03-14")
 	)
