File: BoardDesigns/TagPwrMonitor/TagPwrMonitor.kicad_pcb (KiCad board)
At the start: 2 copper layers, 51 x 60 mm, 16 parts, among them J1 JST XH_B4B-XH, J101 Conn_02x03_Odd_Even, J102 Conn_01x04_Female, U1 XC6206PxxxMR, U2 SN74LV1T04DBVR

Commit message: checkpoint
Parts:
- removed JP1, JP2, JP3: SolderJumper_2_Bridged, Jumper:SolderJumper-2_P1.3mm_Open_RoundedPad1.0x1.5mm
- added C3: 100nf, Capacitor_SMD:C_0805_2012Metric, F.Cu at (119.5, 79.4)
- added J2: Conn_01x03, Connector_PinHeader_2.54mm:PinHeader_1x03_P2.54mm_Vertical, F.Cu at (140.4, 70.8)
- J102: value Conn_01x04_Female -> swd connector
- R2: value 2.2k -> 10k
- R3: value 2.2k -> 1k
- moved C1 2.95 mm to (143.7, 74.7)
- moved C2 2.95 mm to (148.1, 78.4)
- moved U1 2.95 mm to (148.2, 74.8)
- moved R3 2.01 mm to (115.8, 82.9)
- moved R2 2.01 mm to (123.1, 83.8)
- moved U2 2.01 mm to (119.5, 82.8)
Connections:
- C2 pad 1: Net-(JP2-B) -> /TAG_MIRROR
- U1 pad 3: Net-(JP2-B) -> /TAG_MIRROR
Routing:
- net /EXT_PWR: track 29.6 -> 0.90 mm
- net Net-(JP2-B): track 16.2 -> 0.00 mm
- net /TAG_MIRROR: track 28.1 -> 43.6 mm
- net /NRST: track 9.81 -> 11.9 mm
- net /TAG_RESET: track 21.6 -> 19.7 mm
- net GND: track 4.75 -> 6.17 mm, vias 8 -> 7
- net Net-(J2-Pin_3): track 7.87 -> 7.17 mm
Other:
- board text added: "V1.8"
- board text added: "Vsense"
- board text removed: "JP3 - STLINK Sense = VMirror JP1 & JP2 -- STLINK Sense = 1.8V"
