File: BoardDesigns/TagPwrMonitor/TagPwrMonitor.kicad_sch (KiCad schematic)
At the start: 16 parts, among them J1 JST XH_B4B-XH, J101 Conn_02x03_Odd_Even, J102 Conn_01x04_Female, U1 XC6206PxxxMR, U2 SN74LV1T04DBVR

Commit message: checkpoint
Parts:
- removed JP1, JP2, JP3: SolderJumper_2_Bridged, Jumper:SolderJumper-2_P1.3mm_Open_RoundedPad1.0x1.5mm, symbol Jumper:SolderJumper_2_Bridged
- added C3: 100nf, Capacitor_SMD:C_0805_2012Metric, symbol Device:C
- added J2: Conn_01x03, Connector_PinHeader_2.54mm:PinHeader_1x03_P2.54mm_Vertical, symbol Connector_Generic:Conn_01x03
- J102: value Conn_01x04_Female -> swd connector
- R2: value 2.2k -> 10k; LCSC C17520 -> C17414; MPN 0805W8F2201T5E -> 0805W8F1002T5E
- R3: value 2.2k -> 1k; LCSC C17520 -> C17513; MPN 0805W8F2201T5E -> 0805W8F1001T5E
Connections:
- net GND: now also C3.2
- net STLINK_VSENSE: now also J2.2 (Pin_2)
- net TAG_MIRROR: now also C2.1, U1.3 (VI), C3.1, J2.1 (Pin_1)
- net at C1.1, U1.2 (VO): now also J2.3 (Pin_3)
