File: BoardDesigns/js320-faceplate/js320-faceplate.kicad_pcb (KiCad board)
At the start: 2 copper layers, 95 x 24.7 mm, 20 parts, among them J1 JS220, J3 Conn_01x04_Socket, J4 54-00286, SW1 SS-10-23NPE, U1 LT3045xDD, U2 XC6206PxxxMR, U4 PUCC33420RAQR

Commit message: update faceplate and imutagnand-breakout
Other:
- board text added: "C"
Changed lines of the file:
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@@
 			)
 		)
-		(attr exclude_from_pos_files exclude_from_bom dnp)
+		(attr exclude_from_pos_files exclude_from_bom)
 		(duplicate_pad_numbers_are_jumpers no)
 		(fp_line
@@
 			)
 		)
-		(attr through_hole exclude_from_pos_files exclude_from_bom dnp)
+		(attr through_hole exclude_from_pos_files exclude_from_bom)
 		(duplicate_pad_numbers_are_jumpers no)
 		(fp_line
@@
 		)
 		(embedded_fonts no)
-		(model "/Users/geobrown/Research/tag-designs/hardware/BoardDesigns/libraries/packages3D/SS-10-23NP-LE.stp"
+		(model "${KIPRMOD}/../libraries/packages3D/SS-10-23NP-LE.stp"
 			(offset
 				(xyz 4 -4 6.5)
@@
 		)
 	)
+	(gr_text "C"
+		(at 111.875 81.175 0)
+		(layer "B.SilkS")
+		(effects
+			(font
+				(size 1 1)
+				(thickness 0.15)
+			)
+			(justify left bottom mirror)
+		)
+	)
 	(gr_text "Geoffrey Brown\n6/20/26"
 		(at 138.3 90 0)
@@
 	)
 	(segment
-		(start 162.55 82.049997)
-		(end 163.399997 82.049997)
-		(width 0.1524)
-		(layer "B.Cu")
-		(net "GNDPWR")
-	)
-	(segment
 		(start 163.8 80.6)
 		(end 164.55 80.6)
@@
 	)
 	(segment
+		(start 162.55 82.049997)
+		(end 163.399997 82.049997)
+		(width 0.1524)
+		(layer "B.Cu")
+		(net "GNDPWR")
+	)
+	(segment
 		(start 163.650003 80.749997)
 		(end 163.8 80.6)
@@
 	)
 	(segment
+		(start 163.399997 82.049997)
+		(end 163.4 82.05)
+		(width 0.1524)
+		(layer "B.Cu")
+		(net "GNDPWR")
+	)
+	(segment
 		(start 171.1 80.65)
 		(end 171.15 80.6)
@@
 		(layer "B.Cu")
 		(net "GNDPWR")
-	)
-	(segment
-		(start 163.399997 82.049997)
-		(end 163.4 82.05)
-		(width 0.1524)
-		(layer "B.Cu")
-		(net "GNDPWR")
