File: BoardDesigns/js320-faceplate/js320-faceplate.kicad_sch (KiCad schematic)
At the start: 15 parts, among them J1 JS220, J2 Barrel_Jack, J3 Conn_01x04_Socket, SW1 SS-10-23NP-LE, U1 LT3045xDD, U2 XC6206PxxxMR

Commit message: checkpoint
Parts:
- removed J2: Barrel_Jack, Connector_BarrelJack:BarrelJack_CUI_PJ-063AH_Horizontal_CircularHoles, symbol Connector:Barrel_Jack
- added C10, C7: 22nf, Capacitor_SMD:C_0402_1005Metric, symbol Device:C
- added C8: 22uf, Capacitor_SMD:C_0805_2012Metric, symbol Device:C
- added C9: 10uf, Capacitor_SMD:C_0805_2012Metric, symbol Device:C
- added J4: 54-00286, libraries:TENSILITY_54-00286, symbol tag_library:54-00286
- added U4: PUCC33420RAQR, libraries:VSON-FCRLF12_RAQ_TEX, symbol tag_library:PUCC33420RAQR
- C2: value 4.7uf -> 22nf; footprint Capacitor_SMD:C_0805_2012Metric -> Capacitor_SMD:C_0402_1005Metric; LCSC C1779 -> C1532; MFN Samsung Electro-Mechanics -> FH (Guangdong Fenghua Advanced Tech); MPN CL21A475KAQNNNE -> 0402B223K500NT
- C3: value 4.7uf -> 10uf; LCSC C1779 -> C15850; MPN CL21A475KAQNNNE -> CL21A106KAYNNNE
- R1: value 18K -> 18k
- R2: value 24.9K -> 24k
- R3: value 33K -> 33k
- R4: value 1K -> 1k
- SW1: value SS-10-23NP-LE -> SS-10-23NPE
Connections:
- net GND: now also C10.2, C8.2, U4.10 (GNDS), U4.11 (GNDS), U4.12 (GNDS), U4.9 (GNDS)
- net vin: now also C10.1, C8.1, U4.7 (SEL), U4.8 (VCC)
- new net GNDPWR: C7.2, C9.2, J4.B, U4.3 (GNDP), U4.4 (GNDP), U4.5 (GNDP), U4.6 (GNDP)
- new net VINP: C7.1, C9.1, J4.A, U4.1 (EN/FLT), U4.2 (VINP)
- no-connect marks 5 -> 6
Other:
- moved on the sheet: C1, C4, C5, R4, U1, U2
