File: BoardDesigns/BitPresTag/BitPresTag.kicad_sch (KiCad schematic)
At the start: 23 parts, among them J201 CONN_02X04, J301 Conn_01x01, J302 Conn_01x01, J303 Conn_01x01, J304 Conn_01x01, J401 CONN_01X02, Q501 Q_NPN_BEC, U1 at25ex321D-UUN, U2 adxl362, U3 LPS27HHWTR, U302 stm32l431kc, U501 RV-3028-C7

Commit message: added imutag with bmp581, bitprestag with bmp585
Other:
- note added: "scl and sda are reversed"
Changed lines of the file:
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@@
+		)
+	)
+	(text "scl and sda are reversed"
+		(exclude_from_sim no)
+		(at 123.19 39.116 0)
+		(effects
+			(font
+				(size 1.524 1.524)
+			)
 		)
 	)
