File: BoardDesigns/IMUTagNandBreakcoutv2/IMUTagNandBreakcoutv2.kicad_pcb (KiCad board)
At the start: 4 copper layers, 48.3 x 48.3 mm, 20 parts, among them J3 Conn_01x17, J4 Conn_01x17, U1 TPS22916BYFPR, U2 BMM350, U4 LSM6DSV, U5 LPS22HH, U6 GD5F1GQ5REYFGR

Commit message: added imutag with bmp581, bitprestag with bmp585
Parts:
- added TP1: TestPoint, TestPoint:TestPoint_Pad_D2.0mm, F.Cu at (135.1, 77.7)
- U5: value LPS22HH -> LPS22HHTR
- U6: value GD5F1GQ5REYFGR -> GD5F1GQ5REYIGR
- moved C4 8.26 mm to (131.4, 100.0), turned to 0 degrees
- moved C1 4.60 mm to (132.8, 107.2)
- moved C9 4.60 mm to (131.0, 107.2)
- moved U4 4.60 mm to (131.6, 103.9)
- moved C13 4.43 mm to (133.7, 93.3), turned to -90 degrees
- moved C12 2.58 mm to (129.4, 92.9), turned to 90 degrees
- moved U2 2.05 mm to (131.2, 92.8), turned to 0 degrees
Routing:
- net /BMM_INT: track 30.3 -> 36.3 mm
- net /LSM_TRG: track 40.5 -> 45.7 mm
- net /SDA: track 26.6 -> 31.4 mm
- net /AT25_SCK: track 51.7 -> 56.2 mm
- net /LSM_CS: track 27.3 -> 22.9 mm
- net /AT25_MOSI: track 51.3 -> 55.6 mm
- net /WKUP1: track 23.8 -> 28.0 mm
- net /AT25_MISO: track 48.8 -> 52.7 mm
- net /SCL: track 27.3 -> 30.6 mm
- net /Flash 1V8: track 18.5 -> 21.3 mm
Other:
- board text added: "BMM350 X,Y = Y,X Z=-Z"
- board text added: "LSM_CS"
- board text removed: "BMM350 X=-X Z=-Z"
