File: BoardDesigns/IMUTagNandBreakcoutv2/IMUTagNandBreakcoutv2.kicad_sch (KiCad schematic)
At the start: 20 parts, among them J3 Conn_01x17, J4 Conn_01x17, U1 TPS22916BYFPR, U2 BMM350, U4 LSM6DSV, U5 LPS22HH, U6 GD5F1GQ5REYFGR

Commit message: added imutag with bmp581, bitprestag with bmp585
Parts:
- added TP1: TestPoint, TestPoint:TestPoint_Pad_D2.0mm, symbol Connector:TestPoint
- U1: MANUFACTURER (none) -> Texas Instruments
- U5: value LPS22HH -> LPS22HHTR; MPN LPS22HH -> LPS22HHTR
- U6: value GD5F1GQ5REYFGR -> GD5F1GQ5REYIGR; LCSC C2976330 -> C2927042; MPN GD5F1GQ5REYFGR -> GD5F1GQ5REYIGR
Connections:
- net Flash 1V8: now also TP1.1
Changed lines of the file:
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@@
 	)
 	(junction
+		(at 209.55 88.9)
+		(diameter 0)
+		(color 0 0 0 0)
+	)
+	(junction
 		(at 231.14 152.4)
 		(diameter 0)
@@
 	)
 	(symbol
+		(lib_id "Connector:TestPoint")
+		(at 209.55 88.9 0)
+		(unit 1)
+		(body_style 1)
+		(exclude_from_sim no)
+		(in_bom yes)
+		(on_board yes)
+		(in_pos_files yes)
+		(dnp no)
+		(fields_autoplaced yes)
+		(property "Reference" "TP1"
+			(at 212.09 84.3279 0)
+			(show_name no)
+			(do_not_autoplace no)
+			(effects
+				(font
+					(size 1.27 1.27)
+				)
+				(justify left)
+			)
+		)
+		(property "Value" "TestPoint"
+			(at 212.09 86.8679 0)
+			(show_name no)
+			(do_not_autoplace no)
+			(effects
+				(font
+					(size 1.27 1.27)
+				)
+				(justify left)
+			)
+		)
+		(property "Footprint" "TestPoint:TestPoint_Pad_D2.0mm"
+			(at 214.63 88.9 0)
+			(hide yes)
+			(show_name no)
+			(do_not_autoplace no)
+			(effects
+				(font
+					(size 1.27 1.27)
+				)
+			)
+		)
+		(property "Datasheet" ""
+			(at 214.63 88.9 0)
+			(hide yes)
+			(show_name no)
+			(do_not_autoplace no)
+			(effects
+				(font
+					(size 1.27 1.27)
+				)
+			)
+		)
+		(property "Description" "test point"
+			(at 209.55 88.9 0)
+			(hide yes)
+			(show_name no)
+			(do_not_autoplace no)
+			(effects
+				(font
+					(size 1.27 1.27)
+				)
+			)
+		)
+		(pin "1"
+		)
+		(instances
+			(project "IMUTagNandBreakcoutv2"
+				(path "/dc006d87-46a7-47a2-9c65-845f7016dec0"
+					(reference "TP1")
+					(unit 1)
+				)
+			)
+		)
+	)
+	(symbol
 		(lib_id "power:GND")
 		(at 238.76 116.84 0)
@@
 			)
 		)
-		(property "Value" "LPS22HH"
+		(property "Value" "LPS22HHTR"
 			(at 69.85 176.5299 0)
 			(show_name no)
@@
 			)
 		)
-		(property "MPN" "LPS22HH"
+		(property "MPN" "LPS22HHTR"
 			(at 81.28 176.53 0)
 			(hide yes)
@@
 			)
 		)
-		(property "Value" "GD5F1GQ5REYFGR"
+		(property "Value" "GD5F1GQ5REYIGR"
 			(at 210.82 110.744 0)
 			(show_name no)
@@
 			)
 		)
-		(property "MPN" "GD5F1GQ5REYFGR"
+		(property "MPN" "GD5F1GQ5REYIGR"
 			(at 236.22 102.87 0)
 			(hide yes)
@@
 			)
 		)
-		(property "LCSC" "C2976330"
+		(property "LCSC" "C2927042"
 			(at 236.22 102.87 0)
 			(hide yes)
@@
 			)
 		)
+		(property "MANUFACTURER" "Texas Instruments"
+			(at 191.77 110.49 0)
+			(hide yes)
+			(show_name no)
+			(do_not_autoplace no)
+			(effects
+				(font
+					(size 1.27 1.27)
+				)
+				(justify bottom)
+			)
+		)
