File: BoardDesigns/IMUTagNandBMP581-breakout/IMUTagNandBMP581-breakout.kicad_pcb (KiCad board)
At the start: 4 copper layers, 48.3 x 48.3 mm, 21 parts, among them J3 Conn_01x17, J4 Conn_01x17, U1 TPS22916BYFPR, U2 BMM350, U3 BMP581, U4 LSM6DSV, U6 GD5F1GQ5REYIGR

Commit message: added smps breakout board
Parts:
- U6: value GD5F1GQ5REYIGR -> GD5F2GM7REYIGR
Changed lines of the file:
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@@
 			)
 		)
-		(property "Value" "GD5F1GQ5REYIGR"
+		(property "Value" "GD5F2GM7REYIGR"
 			(at 0 3.95 0)
 			(layer "F.Fab")
@@
 			)
 		)
-		(property "Datasheet" "https://www.mouser.com/datasheet/3/1550/1/DS_00860_GD5F1GM7RE_Rev1.3.pdf"
+		(property "Datasheet" ""
 			(at 0 0 0)
 			(layer "F.Fab")
@@
 			)
 		)
-		(property "MPN" "GD5F1GQ5REYIGR"
+		(property "MPN" "GD5F2GM7REYIGR"
 			(at 0 0 0)
 			(unlocked yes)
@@
 			)
 		)
-		(property "LCSC" "C2927042"
+		(property "LCSC" "C23706308"
 			(at 0 0 0)
 			(unlocked yes)
