File: BoardDesigns/IMUTagNandBMP581-breakout/IMUTagNandBMP581-breakout.kicad_sch (KiCad schematic)
At the start: 21 parts, among them J3 Conn_01x17, J4 Conn_01x17, U1 TPS22916BYFPR, U2 BMM350, U3 BMP581, U4 LSM6DSV, U6 GD5F1GQ5REYIGR

Commit message: added smps breakout board
Parts:
- U6: value GD5F1GQ5REYIGR -> GD5F2GM7REYIGR; LCSC C2927042 -> C23706308; MPN GD5F1GQ5REYIGR -> GD5F2GM7REYIGR
Changed lines of the file:
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@@
 			)
 		)
-		(property "Value" "GD5F1GQ5REYIGR"
+		(property "Value" "GD5F2GM7REYIGR"
 			(at 210.82 110.744 0)
 			(show_name no)
@@
 			)
 		)
-		(property "Datasheet" "https://www.mouser.com/datasheet/3/1550/1/DS_00860_GD5F1GM7RE_Rev1.3.pdf"
+		(property "Datasheet" ""
 			(at 236.22 120.396 0)
 			(hide yes)
@@
 			)
 		)
-		(property "MPN" "GD5F1GQ5REYIGR"
+		(property "MPN" "GD5F2GM7REYIGR"
 			(at 236.22 102.87 0)
 			(hide yes)
@@
 			)
 		)
-		(property "LCSC" "C2927042"
+		(property "LCSC" "C23706308"
 			(at 236.22 102.87 0)
 			(hide yes)
