File: BoardDesigns/tag-breakout-u375-smps-v1/stm32.kicad_sch (KiCad schematic)
At the start: 16 parts, among them J3 Conn_01x17, J4 Conn_01x17, Q1 Q_NPN_BEC, U2 TPS62840YBGR, U3 stm32U375, U6 RV-3028-C7

Commit message: checkpoint
Parts:
- C8: value 4.7uF -> 4.7uf; LCSC C23733 -> C335105; MFN Samsung Electro-Mechanics -> Murata; MPN CL05A475MP5NRNC -> GRM155R61A475MEAAD
Changed lines of the file:
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@@
+	)
+	(symbol
+		(lib_id "power:PWR_FLAG")
+		(at 212.09 74.93 0)
+		(unit 1)
+		(body_style 1)
+		(exclude_from_sim no)
+		(in_bom yes)
+		(on_board yes)
+		(in_pos_files yes)
+		(dnp no)
+		(fields_autoplaced yes)
+		(property "Reference" "#FLG01"
+			(at 212.09 73.025 0)
+			(hide yes)
+			(show_name no)
+			(do_not_autoplace no)
+			(effects
+				(font
+					(size 1.27 1.27)
+				)
+			)
+		)
+		(property "Value" "PWR_FLAG"
+			(at 212.09 69.85 0)
+			(show_name no)
+			(do_not_autoplace no)
+			(effects
+				(font
+					(size 1.27 1.27)
+				)
+			)
+		)
+		(property "Footprint" ""
+			(at 212.09 74.93 0)
+			(hide yes)
+			(show_name no)
+			(do_not_autoplace no)
+			(effects
+				(font
+					(size 1.27 1.27)
+				)
+			)
+		)
+		(property "Datasheet" ""
+			(at 212.09 74.93 0)
+			(hide yes)
+			(show_name no)
+			(do_not_autoplace no)
+			(effects
+				(font
+					(size 1.27 1.27)
+				)
+			)
+		)
+		(property "Description" "Special symbol for telling ERC where power comes from"
+			(at 212.09 74.93 0)
+			(hide yes)
+			(show_name no)
+			(do_not_autoplace no)
+			(effects
+				(font
+					(size 1.27 1.27)
+				)
+			)
+		)
+		(pin "1"
+		)
+		(instances
+			(project "tag-breakout-u375-smps-v1"
+				(path "/2d561ecb-394a-4bb7-a154-94e4285b4f36/00000000-0000-0000-0000-00005fa00cea"
+					(reference "#FLG01")
+					(unit 1)
+				)
+			)
+		)
 	)
 	(symbol
@@
 			)
 		)
-		(property "Value" "4.7uF"
+		(property "Value" "4.7uf"
 			(at 59.69 40.6399 0)
 			(show_name no)
@@
 			)
 		)
-		(property "LCSC" "C23733"
+		(property "LCSC" "C335105"
 			(at 55.88 39.37 0)
 			(hide yes)
@@
 			)
 		)
-		(property "MFN" "Samsung Electro-Mechanics"
+		(property "MFN" "Murata"
 			(at 55.88 39.37 0)
 			(hide yes)
@@
 			)
 		)
-		(property "MPN" "CL05A475MP5NRNC"
+		(property "MPN" "GRM155R61A475MEAAD"
 			(at 55.88 39.37 0)
 			(hide yes)

Commit message: U375 smps breakout and UIUC breakout
Parts:
- L1: footprint Inductor_SMD:L_Murata_DFE201610P -> project_library:IND_DFE2016_MUR
Changed lines of the file:
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@@
 			)
 		)
-		(property "Footprint" "Inductor_SMD:L_Murata_DFE201610P"
+		(property "Footprint" "project_library:IND_DFE2016_MUR"
 			(at 203.2 69.85 0)
 			(hide yes)
