File: BoardDesigns/tag-breakout-u375-smps-v1/tag-breakout-u375-smps-v1.kicad_pcb (KiCad board)
At the start: 4 copper layers, 53.3 x 73.7 mm, 51 parts, among them J1 Conn_01x04_Female, J102 Conn_02x05_Odd_Even, J104 USB_B_Mini, J2 Conn_01x02_Male, J3 Conn_01x17, J4 Conn_01x17, Q1 Q_NPN_BEC, SW2 SW_SPDT, U1 XC6206, U10 AP2112K-1.8, U105 Tactile Switch, U2 TPS62840YBGR, U3 stm32U375, U4 USBLC6-2P6, U5 STM32L432KBU6, U6 RV-3028-C7, U7 SN74LVC1T45DCK, U8 SN74LVC1T45DCK

Commit message: checkpoint
Parts:
- C8: value 4.7uF -> 4.7uf
- D1: value LED-GREEN -> LED
- D105: value LED-RED -> LED
- moved U2 3.09 mm to (137.6, 81.7)
- moved C4 2.97 mm to (139.7, 81.7)
- moved L1 2.83 mm to (138.5, 84.1)
- moved C10 2.82 mm to (138.1, 80.0)
Routing:
- net TAG_3V3: track 0.00 -> 8.89 mm
- net GND: track 55.2 -> 58.0 mm, vias 49 -> 52
- net Net-(U2-SW): track 0.00 -> 2.25 mm
- net TAG_1V8: track 10.6 -> 12.4 mm, vias 4 -> 5
- added copper zone on F.Cu, net Net-(U2-SW)
- added copper zone on F.Cu, net TAG_1V8
- added copper zone on F.Cu, net TAG_3V3
Other:
- board text added: "BitTag Breakout U375 SMPS 1v8"
- board text added: "Geoffrey Brown 8/19/26"
- board text added: "MIR."
- board text added: "PWR"
- board text removed: "BitTag Breakout U375 1v8 V2"
- board text removed: "Geoffrey Brown 7/28/26"

Commit message: U375 smps breakout and UIUC breakout
Parts:
- L1: footprint Inductor_SMD:L_Murata_DFE201610P -> project_library:IND_DFE2016_MUR
Changed lines of the file:
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@@
 			)
 		)
+		(property "FT Rotation Offset" "-90"
+			(at 0 0 0)
+			(unlocked yes)
+			(layer "F.Fab")
+			(hide yes)
+			(effects
+				(font
+					(size 1 1)
+					(thickness 0.15)
+				)
+			)
+		)
 		(sheetname "/stm32/")
 		(sheetfile "stm32.kicad_sch")
@@
 		)
 	)
-	(footprint "Inductor_SMD:L_Murata_DFE201610P"
+	(footprint "project_library:IND_DFE2016_MUR"
 		(layer "F.Cu")
 		(at 138.475 84.1 180)
-		(descr "Inductor, Murata, DFE201610P, 2.0x1.6x1.0mm, (https://www.murata.com/~/media/webrenewal/products/inductor/chip/tokoproducts/wirewoundmetalalloychiptype/m_dfe201610p.ashx)")
-		(tags "power chip flatwire")
+		(tags "DFE201612E-2R2M=P2 ")
 		(property "Reference" "L1"
-			(at 0 -1.75 0)
+			(at 2.775 -0.05 0)
+			(unlocked yes)
 			(layer "F.SilkS")
-			(hide yes)
 			(effects
 				(font
@@
 		)
 		(property "Value" "2.2uH"
-			(at 0 1.75 0)
+			(at 0 0 180)
+			(unlocked yes)
 			(layer "F.Fab")
 			(effects
@@
 		)
 		(property "Datasheet" ""
-			(at 0 0 0)
+			(at 0 0 180)
 			(layer "F.Fab")
 			(hide yes)
@@
 		)
 		(property "Description" "Inductor"
-			(at 0 0 0)
+			(at 0 0 180)
 			(layer "F.Fab")
 			(hide yes)
@@
 			)
 		)
-		(property "KiLib_Generator" "inductor/SMD"
-			(at 0 0 0)
-			(layer "F.SilkS")
-			(hide yes)
-			(effects
-				(font
-					(size 1 1)
-					(thickness 0.15)
-				)
-			)
-		)
 		(property "MFN" "Murata"
 			(at 0 0 180)
@@
 		(attr smd)
 		(duplicate_pad_numbers_are_jumpers no)
-		(fp_line
-			(start 1.11 1.06)
-			(end -1.11 1.06)
+		(fp_circle
+			(center -2.2987 0)
+			(end -2.2225 0)
 			(stroke
-				(width 0.12)
+				(width 0.1524)
 				(type solid)
 			)
+			(fill no)
 			(layer "F.SilkS")
 		)
 		(fp_line
-			(start -1.11 -1.06)
-			(end 1.11 -1.06)
+			(start 1.7145 1.1557)
+			(end -1.7145 1.1557)
 			(stroke
-				(width 0.12)
+				(width 0.1524)
 				(type solid)
 			)
-			(layer "F.SilkS")
+			(layer "F.CrtYd")
 		)
-		(fp_rect
-			(start -1.25 -1.05)
-			(end 1.25 1.05)
+		(fp_line
+			(start 1.7145 -1.1557)
+			(end 1.7145 1.1557)
 			(stroke
-				(width 0.05)
+				(width 0.1524)
 				(type solid)
 			)
-			(fill no)
 			(layer "F.CrtYd")
 		)
-		(fp_rect
-			(start -1 -0.8)
-			(end 1 0.8)
+		(fp_line
+			(start -1.7145 1.1557)
+			(end -1.7145 -1.1557)
 			(stroke
-				(width 0.1)
+				(width 0.1524)
+				(type solid)
+			)
+			(layer "F.CrtYd")
+		)
+		(fp_line
+			(start -1.7145 -1.1557)
+			(end 1.7145 -1.1557)
+			(stroke
+				(width 0.1524)
+				(type solid)
+			)
+			(layer "F.CrtYd")
+		)
+		(fp_line
+			(start 1.1049 0.9017)
+			(end 1.1049 -0.9017)
+			(stroke
+				(width 0.0254)
+				(type solid)
+			)
+			(layer "F.Fab")
+		)
+		(fp_line
+			(start 1.1049 0.9017)
+			(end 1.1049 -0.9017)
+			(stroke
+				(width 0.0254)
+				(type solid)
+			)
+			(layer "F.Fab")
+		)
+		(fp_line
+			(start 1.1049 -0.9017)
+			(end 0.2921 -0.9017)
+			(stroke
+				(width 0.0254)
+				(type solid)
+			)
+			(layer "F.Fab")
+		)
+		(fp_line
+			(start 1.1049 -0.9017)
+			(end -1.1049 -0.9017)
+			(stroke
+				(width 0.0254)
+				(type solid)
+			)
+			(layer "F.Fab")
+		)
+		(fp_line
+			(start 0.2921 0.9017)
+			(end 1.1049 0.9017)
+			(stroke
+				(width 0.0254)
+				(type solid)
+			)
+			(layer "F.Fab")
+		)
+		(fp_line
+			(start 0.2921 -0.9017)
+			(end 0.2921 0.9017)
+			(stroke
+				(width 0.0254)
+				(type solid)
+			)
+			(layer "F.Fab")
+		)
+		(fp_line
+			(start -0.2921 0.9017)
+			(end -0.2921 -0.9017)
+			(stroke
+				(width 0.0254)
+				(type solid)
+			)
+			(layer "F.Fab")
+		)
+		(fp_line
+			(start -0.2921 -0.9017)
+			(end -1.1049 -0.9017)
+			(stroke
+				(width 0.0254)
+				(type solid)
+			)
+			(layer "F.Fab")
+		)
+		(fp_line
+			(start -1.1049 0.9017)
+			(end 1.1049 0.9017)
+			(stroke
+				(width 0.0254)
+				(type solid)
+			)
+			(layer "F.Fab")
+		)
+		(fp_line
+			(start -1.1049 0.9017)
+			(end -0.2921 0.9017)
+			(stroke
+				(width 0.0254)
+				(type solid)
+			)
+			(layer "F.Fab")
+		)
+		(fp_line
+			(start -1.1049 -0.9017)
+			(end -1.1049 0.9017)
+			(stroke
+				(width 0.0254)
+				(type solid)
+			)
+			(layer "F.Fab")
+		)
+		(fp_line
+			(start -1.1049 -0.9017)
+			(end -1.1049 0.9017)
+			(stroke
+				(width 0.0254)
+				(type solid)
+			)
+			(layer "F.Fab")
+		)
+		(fp_circle
+			(center -0.7493 0)
+			(end -0.6731 0)
+			(stroke
+				(width 0.0254)
 				(type solid)
 			)
@@
 		)
 		(fp_text user "${REFERENCE}"
-			(at 0 0 0)
+			(at 0 0 180)
+			(unlocked yes)
 			(layer "F.Fab")
 			(effects
 				(font
-					(size 0.5 0.5)
-					(thickness 0.08)
+					(size 1 1)
+					(thickness 0.15)
 				)
 			)
 		)
-		(pad "1" smd roundrect
-			(at -0.725 0 180)
-			(size 0.55 1.6)
+		(pad "1" smd rect
+			(at -0.8763 0 180)
+			(size 1.1684 1.8034)
 			(layers "F.Cu" "F.Mask" "F.Paste")
-			(roundrect_rratio 0.25)
 			(net "TAG_1V8")
 			(pinfunction "1_1")
 			(pintype "passive")
 		)
-		(pad "2" smd roundrect
-			(at 0.725 0 180)
-			(size 0.55 1.6)
+		(pad "2" smd rect
+			(at 0.8763 0 180)
+			(size 1.1684 1.8034)
 			(layers "F.Cu" "F.Mask" "F.Paste")
-			(roundrect_rratio 0.25)
 			(net "Net-(U2-SW)")
 			(pinfunction "2_2")
 			(pintype "passive")
 		)
-		(embedded_fonts no)
-		(model "${KICAD10_3DMODEL_DIR}/Inductor_SMD.3dshapes/L_Murata_DFE201610P.step"
-			(offset
-				(xyz 0 0 0)
-			)
-			(scale
-				(xyz 1 1 1)
-			)
-			(rotate
-				(xyz 0 0 0)
+		(zone
+			(layer "F.Cu")
+			(hatch full 0.508)
+			(connect_pads
+				(clearance 0)
+			)
+			(min_thickness 0.254)
+			(keepout
+				(tracks not_allowed)
+				(vias not_allowed)
+				(pads allowed)
+				(copperpour not_allowed)
+				(footprints allowed)
+			)
+			(placement
+				(enabled no)
+				(sheetname "")
+			)
+			(fill
+				(thermal_gap 0.508)
+				(thermal_bridge_width 0.508)
+				(island_removal_mode 0)
+			)
+			(polygon
+				(pts
+					(xy 138.7163 84.9509) (xy 138.2337 84.9509) (xy 138.2337 83.2491) (xy 138.7163 83.2491)
+				)
 			)
 		)
+		(embedded_fonts no)
 	)
 	(footprint "Resistor_SMD:R_0402_1005Metric"
@@
 			(unlocked yes)
 			(layer "F.Fab")
+			(hide yes)
+			(effects
+				(font
+					(size 1 1)
+					(thickness 0.15)
+				)
+			)
+		)
+		(property "FT Rotation Offset" "180"
+			(at 0 0 0)
+			(unlocked yes)
+			(layer "F.Fab")
