File: BoardDesigns/tag-breakout-u375-smps-v1/tag-breakout-u375-smps-v1.kicad_sch (KiCad schematic)
At the start: 35 parts, among them J1 Conn_01x04_Female, J102 Conn_02x05_Odd_Even, J104 USB_B_Mini, J2 Conn_01x02_Male, SW2 SW_SPDT, U1 XC6206, U10 AP2112K-1.8, U105 Tactile Switch, U4 USBLC6-2P6, U5 STM32L432KBU6, U7 SN74LVC1T45DCK, U8 SN74LVC1T45DCK

Commit message: checkpoint
Parts:
- D1: value LED-GREEN -> LED
- D105: value LED-RED -> LED
Changed lines of the file:
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@@
 			)
 		)
-		(property "Value" "LED-RED"
+		(property "Value" "LED"
 			(at 55.88 120.65 0)
 			(show_name no)
@@
 			)
 		)
-		(property "Value" "LED-GREEN"
+		(property "Value" "LED"
 			(at 38.1 120.65 0)
 			(show_name no)

Commit message: checkpoint
Other:
- title: Tag  stm32u375 v2 -> Tag  stm32u375 smps
Changed lines of the file:
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@@
 	(paper "USLetter")
 	(title_block
-		(title "Tag  stm32u375 v2")
-		(date "2026-07-28")
+		(title "Tag  stm32u375 smps")
+		(date "2026-08-30")
 	)
 	(text "5 Pin package but pin 4 is defined\nas NC in datasheet"
