File: BoardDesigns/BitPresTagBMP581/BitPresTagBMP581.kicad_sch (KiCad schematic)
At the start: 26 parts, among them J201 CONN_02X04, J301 Conn_01x01, J302 Conn_01x01, J303 Conn_01x01, J304 Conn_01x01, J401 CONN_01X02, Q501 Q_NPN_BEC, U1 at25ex321D-UUN, U2 ADXL367BCCZ-RL7, U3 BMP585, U302 stm32l431kc, U501 RV-3028-C8

Commit message: added smps breakout board
Parts:
- C1, C7: LCSC (none) -> C181047; MFN (none) -> Murata; MPN CL05F104ZO5NNNC -> GRM033C81E104KE14D
- C2: DISTPN 490-7229-2-ND -> (none); LCSC C76929 -> C181047; MFN murata -> Murata; MPN GRM033R60J105MEA2D -> GRM033C81E104KE14D
- C3, C5: LCSC (none) -> C181047
- C501, C502, C503, C504: MPN C181047 -> GRM033C81E104KE14D
- C6: LCSC (none) -> C2185054
- Q501: value Q_NPN_BEC -> PMBT2222AMBYL; DISTPN 1727-2632-1-ND -> (none); LCSC C686658 -> C552701; MPN BC847AMB,315 -> PMBT2222AMBYL
- U2: LCSC (none) -> C17643415; MFN (none) -> Analog Devices; MPN (none) -> ADXL367BCCZ-RL7
- U3: LCSC (none) -> C18184976; MFN (none) -> Bosch; MPN (none) -> BMP585
- U501: value RV-3028-C8 -> RV-3028-C8-32.768kHz-1PPM-TA-QC; LCSC (none) -> C46471039; MPN (none) -> RV-3028-C8-32.768kHz-1PPM-TA-QC
Connections:
- no-connect marks 8 -> 6

Commit message: checkpoint
Other:
- title: BitTag with External Memory and LPS27 -> BitTag with External Memory and BMP585
Changed lines of the file:
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@@
 	(paper "USLetter")
 	(title_block
-		(title "BitTag with External Memory and LPS27")
-		(date "2025-04-25")
+		(title "BitTag with External Memory and BMP585")
+		(date "2026-08-19")
 		(company "IUCS")
 		(comment 1 "Geoffrey Brown")
-		(comment 3 "checked pinouts 4/25/25")
 	)
 	(text "Note: PA15 and PB4 pulled up on reset !"

Commit message: checkpoint
Connections:
- net lps_rdy: now reaches U302.12 (PA6)
- net lps_rdy: now also U3.5 (INT)
- no-connect marks 6 -> 10
Changed lines of the file:
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@@
+	)
+	(no_connect
+		(at 153.67 91.44)
+	)
+	(no_connect
+		(at 153.67 93.98)
 	)
 	(no_connect
@@
 	)
 	(no_connect
+		(at 120.65 119.38)
+	)
+	(no_connect
+		(at 153.67 88.9)
+	)
+	(no_connect
 		(at 87.63 81.28)
 	)
@@
 		)
 	)
+	(label "lps_rdy"
+		(at 118.11 119.38 270)
+		(effects
+			(font
+				(size 1.524 1.524)
+			)
+			(justify right bottom)
+		)
+	)
 	(label "ACCEL_SCK"
 		(at 113.03 119.38 270)
@@
 		)
 	)
+	(label "lps_rdy"
+		(at 210.82 143.51 0)
+		(effects
+			(font
+				(size 1.524 1.524)
+			)
+			(justify left bottom)
+		)
+	)
