File: BoardDesigns/BitPresTagBMP581/BitPresTagBMP581.kicad_sch (KiCad schematic)
At the start: 26 parts, among them J201 CONN_02X04, J301 Conn_01x01, J302 Conn_01x01, J303 Conn_01x01, J304 Conn_01x01, J401 CONN_01X02, Q501 PMBT2222AMBYL, U1 at25ex321D-UUN, U2 ADXL367BCCZ-RL7, U3 BMP585, U302 stm32l431kc, U501 RV-3028-C8-32.768kHz-1PPM-TA-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

Commit message: BitPresTagBMP581: design review, and fix the two defects it found
Full kicad-happy review against a fresh analyzer run. The pre-existing
analysis/ was poisoned (project_settings.source named
BitTagNG-LIS2DU12.kicad_pcb-back.kicad_pro, so every rule-derived number
was measured against the wrong rule set); those three flat JSONs are
removed and the run redone.

Design fixes:
  - C8 220nF on U2.9 VREG_OUT. The ADXL367 datasheet requires an external
    0.2uF on this pin; it was a single-pin net.
  - R2 10R in series in the BMP585 supply (PB1 -> R2 -> C3/C5/U3.4/U3.8).
    BMP585 Table 4 footnote a makes this normative: "For supply ramps
    < 0.01 ms, a 10 Ohm resistor must be connected in series to the power
    supply". Decoupling stays on the load side.
  - U3 pin 9 (L/M) no-connect flag. It is the lasermarking pad; the
    datasheet says no external connection is possible (S/R coverage).
  - U2 pins 7/11 GND pin type power_out -> power_in.
  - Rail relabelled +2V5 -> VCC. There is no 2.5V regulator; the rail is
    VBAT less a Schottky drop and tracks the cell (~3.1V to ~1.9V). VIN
    global labels kept as the environment-facing alias, so the netlist and
    PCB net name are unchanged.

Design rules tightened: edge clearance 0 -> 0.3mm, annular ring 0.1016 ->
0.1524mm, vias 0.5048/0.2mm, and track_not_centered_on_via re-enabled.

Verified: KiCad DRC 0 violations / 0 unconnected, KiCad ERC 0 violations
(was 6), padnet_crosscheck 28 footprints / 0 mismatches. Pinouts verified
against manufacturer PDFs for Q501 (PMBT2222AMB), U1 (AT25XE321D 12-ball
WLCSP), U2 (ADXL367), U3 (BMP585) and U501 (RV-3028 backup network).

.kicad-happy.json rewritten: the previous one had been copied from a
CompassTag-style board and described an AK09940A, a TPS7A2018 at U4 and a
+1V8 rail, none of which exist here. It now carries the real 33-entry pin
map, 21 evidence-backed suppressions and the firmware contracts.

Co-Authored-By: Claude Opus 5 (1M context) <noreply@anthropic.com>
Parts:
- added C8: 220nf, AccelTag:C_0201_0603Metric, symbol Device:C
- added R2: 10, AccelTag:R_0201_0603Metric, symbol Device:R
Connections:
- net GND: now also C8.2
- net LPS_PWR: now also R2.2; no longer C3.1, C5.1, U3.4 (VDDIO), U3.8 (VDD)
- net at U2.9 (VREG_OUT): now also C8.1
- net +2V5 renamed VCC
- new net: C3.1, C5.1, R2.1, U3.4 (VDDIO), U3.8 (VDD)
Other:
- moved on the sheet: C1, C7
