File: BoardDesigns/UIUCBreakout/UIUCBreakout.kicad_pcb (KiCad board)
At the start: 4 copper layers, 48.3 x 48.3 mm, 10 parts, among them J3 Conn_01x17, J4 Conn_01x17, U1 AT25FF321A-SHN-B, U2 ADXL367BCCZ-RL7, U3 BMP585

Commit message: checkpoint
Connections:
- J3 pad 14: unconnected-(J3-Pin_14-Pad14) -> /LPS_RDY
- U3 pad 5: unconnected-(U3-INT-Pad5) -> /LPS_RDY
Routing:
- net /LPS_RDY: track 0.00 -> 22.0 mm, vias 0 -> 1
Other:
- board text added: "PA6 LPS_RDY"
- board text removed: "PA6"
Changed lines of the file:
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@@
 			(size 0.8382 0.6096)
 			(layers "F.Cu" "F.Mask" "F.Paste")
-			(net "unconnected-(U3-INT-Pad5)")
+			(net "/LPS_RDY")
 			(pinfunction "INT_5")
-			(pintype "output+no_connect")
+			(pintype "output")
 		)
 		(pad "6" smd rect
@@
 			(layers "*.Cu" "*.Mask")
 			(remove_unused_layers no)
-			(net "unconnected-(J3-Pin_14-Pad14)")
+			(net "/LPS_RDY")
 			(pinfunction "Pin_14_14")
-			(pintype "passive+no_connect")
+			(pintype "passive")
 		)
 		(pad "15" thru_hole oval
@@
 		)
 	)
-	(gr_text "PA6"
+	(gr_text "PA6 LPS_RDY\n"
 		(at 109.22 109.22 0)
 		(layer "F.SilkS")
@@
 		(net "/AT25_SCK")
 	)
+	(segment
+		(start 126.8016 104.477)
+		(end 125.34 104.477)
+		(width 0.1524)
+		(layer "F.Cu")
+		(net "/LPS_RDY")
+	)
+	(segment
+		(start 125.34 104.477)
+		(end 125.29 104.427)
+		(width 0.1524)
+		(layer "F.Cu")
+		(net "/LPS_RDY")
+	)
+	(via
+		(at 125.29 104.427)
+		(size 0.6096)
+		(drill 0.3)
+		(layers "F.Cu" "B.Cu")
+		(net "/LPS_RDY")
+	)
+	(segment
+		(start 111.6 104.427)
+		(end 106.807 109.22)
+		(width 0.1524)
+		(layer "B.Cu")
+		(net "/LPS_RDY")
+	)
+	(segment
+		(start 125.29 104.427)
+		(end 111.6 104.427)
+		(width 0.1524)
+		(layer "B.Cu")
+		(net "/LPS_RDY")
+	)
 	(zone
