File: BoardDesigns/UIUCBreakout/UIUCBreakout.kicad_sch (KiCad schematic)
At the start: 10 parts, among them J3 Conn_01x17, J4 Conn_01x17, U1 AT25FF321A-SHN-B, U2 ADXL367BCCZ-RL7, U3 BMP585

Commit message: checkpoint
Connections:
- net LPS_RDY: now reaches J3.14 (Pin_14)
- net LPS_RDY: now also U3.5 (INT)
- no-connect marks 21 -> 19
Changed lines of the file:
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@@
-	)
-	(no_connect
-		(at 222.25 99.06)
 	)
 	(no_connect
@@
 	(no_connect
 		(at 123.19 33.02)
-	)
-	(no_connect
-		(at 96.52 53.34)
 	)
 	(no_connect
@@
 		)
 	)
+	(label "LPS_RDY"
+		(at 222.25 99.06 0)
+		(effects
+			(font
+				(size 1.27 1.27)
+			)
+			(justify left bottom)
+		)
+	)
 	(label "LPS_CS"
 		(at 96.52 58.42 180)
 		(effects
 			(font
+				(size 1.27 1.27)
+			)
+			(justify right bottom)
+		)
+	)
+	(label "LPS_RDY"
+		(at 96.52 53.34 180)
+		(effects
+			(font
