File: BoardDesigns/UIUCBreakout/UIUCBreakout.kicad_sch (KiCad schematic)
At the start: 10 parts, among them J3 Conn_01x17, J4 Conn_01x17, U1 AT25FF321A-SHN-B, U2 ADXL367BCCZ-RL7, U3 BMP585

Commit message: UIUCBreakout: add R1/C4, tighten design rules, regenerate 4-layer fab package
Adds the two parts the board was missing:

- R1 (10 R) in series in the BMP585 supply. This is the Bosch-required
  inrush limiter from BMP585 datasheet 6.2.5 Fig. 27, and it sits in the
  power path -- without it U3 is unpowered. Same role as R2 on
  BitPresTagBMP585.
- C4 (0.22 uF) on the ADXL367 VREG_OUT pin. Required, not optional:
  ADXL367 datasheet Table 9 note 1 asks for an external 0.2 uF.

Design rules were on loose defaults (min annular 0.05 mm, edge clearance
0.075 mm). Replaced with the real rule set: 0.1016 mm clearance and track,
0.3 mm copper-to-edge, 0.1524 mm via annular, and explicit via classes
(0.5048/0.2 and 0.61/0.3).

The previously committed jlcpcb/gerber/ set was a 2-layer plot of a
4-layer board -- no CuIn1/CuIn2. That was not cosmetic: J3.7 and J4.1
have no on-layer track and reach +3.3V only through the In1 plane, so
that set would have fabricated a board with no power. Both inner layers
are now present and committed.

Drops the 2026-08-20 production/ export, which predates R1 and C4 and so
carried a BOM and CPL that would have left both unplaced.

Verified against the committed state:

- DRC in place with --refill-zones: 0 violations, 0 unconnected
- Gerbers vs saved board: 114/114 track starts match on CuTop+CuBottom;
  CuIn1/CuIn2 carry real geometry (2863 / 2642 coordinates). Checked by
  geometry, not mtime -- the board is 3 min newer than the export because
  exporting marks it dirty.
- Drill reconciliation: 59 = 59 (0.2 mm x3, 0.3 mm x22 vias, 1.0 mm x34
  header pins; NPTH empty)
- U1 is AT25FF321A-SHN-B, the 208-mil wide EIAJ SOIC. Footprint
  SOIC-8_5.3x6.2mm_P1.27mm is KiCad's JEITA/EIAJ 08-001-BBA 208-mil
  pattern and LCSC C5591126 is package SOIC-8-208mil. Correct pairing;
  the 150-mil part is -SSHN-B / C7455378.

Co-Authored-By: Claude Opus 5 (1M context) <noreply@anthropic.com>
Parts:
- added C4: C, Capacitor_SMD:C_0603_1608Metric, symbol Device:C
- added R1: 10, libraries:R_0603_1608Metric, symbol Device:R
Connections:
- net GND: now also C4.2
- net LPS_PWR: now also R1.1; no longer J4.16 (Pin_16)
- net at U2.9 (VREG_OUT): now also C4.1
- new net LPS_PWR_IN: J4.16 (Pin_16), R1.2
- no-connect marks 19 -> 18
Other:
- title: UIUC Breakout -> UIUC Breakout V2
- moved on the sheet: C1, C3, C5, C7, U3

Commit message: UIUCBreakout: close out the review -- L1-L6 fixed, M3 accepted, L4 withdrawn
Board changes: C6 (4.7 uF) bulk added on +3.3V, 4.12 mm from U1.8; C4 Value
corrected to 0.22uf; U2 ADXL367 symbol refreshed from tag_library; PWR_FLAG
count 1 -> 3; silkscreen at J3.3/J3.4 relabelled PB7/PB6; back-silk date and
the J4.16 LPS_PWR_IN label corrected.

ERC goes from 8 violations to 2 warnings, 0 errors.

M3 -- accepted as-is, do not re-raise. U1 SIO2/SIO3 stay hard-tied to +3.3V
rather than pulled up. The tag has no room for the two resistors, and this
breakout is the preferred place for a quad-mode failure to happen: U1 here is
an 8-lead SOIC that can be desoldered and replaced by hand, where the tag's
WLCSP cannot. That is a better position than the review took -- it converts an
untestable hazard on the tag into a cheap, observable one here. The two
pin_to_pin ERC warnings on U1.3/U1.7 are therefore permanent and expected; they
are inherent to tying bidirectional pins to a net carrying a PWR_FLAG and
cannot be cleared by relocating the flag, since ERC evaluates net-wide.

L4 -- withdrawn, raised in error. The review claimed C7 sat 10.7 mm from the
flash it decouples. C7 is U2's cap, 1.61 mm from the ADXL367 VS pin; the flash
has C2 at 2.42 mm. Capacitors had been paired to parts by reading reference
designators instead of measuring. Measured nearest same-net cap per supply pin:
U1 VCC/C2 2.42, U2 VS/C7 1.61, U2 VDDIO/C1 1.89, U2 VREG_OUT/C4 1.97,
U3 VDD/C5 1.78, U3 VDDIO/C3 1.71 mm -- every supply pin within 2.73 mm. Only
the bulk half of the finding stood, and C6 addresses it.

L1 -- the baseboard fault is a WIRING error, not a naming error, and the
distinction decides the label. /stm32/rtc_scl really does carry the RV-3028's
SCL; what is crossed is which MCU pin it landed on (PB7, which is I2C1_SDA).
Checked against the Micro Crystal RV-3028-C7 Application Manual section 2.2
(pin 3 = SCL, pin 4 = SDA) rather than the KiCad symbol -- a mislabelled symbol
would have inverte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
Parts:
- added C6: 4.7uf, Capacitor_SMD:C_0603_1608Metric, symbol Device:C
- C4: value C -> 0.22uf
Connections:
- net +3.3V: now also C6.1
- net GND: now also C6.2
Other:
- moved on the sheet: C2
