File: BoardDesigns/tagbase-lipo-v1/tagbase-lipo-v1.kicad_sch (KiCad schematic)
At the start: 38 parts, among them J1 Conn_01x04_Female, J101 Conn_02x03_Odd_Even, J102 Conn_02x05_Odd_Even, J104 USB_B_Mini, J2 Conn_01x06, J5 Conn_01x02, SW1 SW_SPDT, SW2 SW_SPDT, U1 XC6206P332MR, U105 Tactile Switch, U2 XC6808ANC28R-G, U3 XC6206P182MR, U4 STM32C071GBUx, U5 SN74LVC1T45DCK, U6 SN74LVC1T45DCK

Commit message: added imutag with bmp581, bitprestag with bmp585
Parts:
- removed C101: 0.1uF, Capacitor_SMD:C_0402_1005Metric, symbol Device:C
- removed C6: 4.7uf, Capacitor_SMD:C_0402_1005Metric, symbol Device:C
- removed D105: LED-GREEN, Diode_SMD:D_0805_2012Metric, symbol Device:LED
- removed H1, H2, H3, H4: MountingHole, MountingHole:MountingHole_2.5mm, symbol Mechanical:MountingHole
- removed J2: Conn_01x06, tagbase:JST_B6B-ZR(LF)(SN), symbol Connector_Generic:Conn_01x06
- removed R5: 100, Resistor_SMD:R_0603_1608Metric, symbol Device:R
- removed U4: STM32C071GBUx, Package_DFN_QFN:QFN-28_4x4mm_P0.5mm, symbol MCU_ST_STM32C0:STM32C071GBUx
- removed U5, U6: SN74LVC1T45DCK, Package_TO_SOT_SMD:SOT-363_SC-70-6, symbol Logic_LevelTranslator:SN74LVC1T45DCK
- added C102, C103, C109, C110, C111, C3, C7, C8: 0.1uF, Capacitor_SMD:C_0402_1005Metric, symbol Device:C
- added R105: 12K, Resistor_SMD:R_0402_1005Metric, symbol Device:R
- added R106: 100, Resistor_SMD:R_0402_1005Metric, symbol Device:R
- added U4: USBLC6-2P6, Package_TO_SOT_SMD:SOT-666, symbol Power_Protection:USBLC6-2P6
- added U5: STM32L432KBU6, Package_DFN_QFN:UFQFPN-32-1EP_5x5mm_P0.5mm_EP3.5x3.5mm, symbol tag-library:stm32l432
- added U7, U8: SN74LVC1T45DCK, Package_TO_SOT_SMD:SOT-363_SC-70-6, symbol Logic_LevelTranslator:SN74LVC1T45DCK
- R102: value 100 -> 220
- R4: footprint Resistor_SMD:R_0603_1608Metric -> Resistor_SMD:R_0402_1005Metric; LCSC C22775 -> C25076; MFN Uniroyal Elec. -> Uniroyal Elec; MPN 0603WAF1000T5E -> 0402WGF1000TCE
Connections:
- net +1V8: now also C103.1, C109.1, U7.6 (VCCB), U8.6 (VCCB)
- net +3V3: now also C4.1, U3.3 (VI), C110.1, C111.1, C3.1, C8.1, U5.1 (VDD), U5.17 (VDD), U5.5 (VDDA/VREF+), U7.1 (VCCA), U7.5 (DIR), U8.1 (VCCA)
- net CSO: now also U5.6 (PA0)
- net GND: now also C102.2, C103.2, C109.2, C110.2, C111.2, C3.2, C7.2, C8.2, R105.1, U4.2 (GND), U5.16 (VSS), U5.32 (VSS), U5.33 (GND), U7.2 (GND), U8.2 (GND)
- net LED_GREEN: now also U5.8 (PA2)
- net LED_RED: now also U5.9 (PA3)
- net NRST: now also C7.1, U5.4 (~{NRST})
- net SWDIO: now also U5.23 (PA13)
- net TAG_RESET: now also R104.2; no longer R104.1
- net TAG_SCK: now also U7.4 (B)
- net TAG_SWDIO: now also R106.2
- net UART_TX: now also U5.19 (PA9)
- net USB_DM: now also U4.4 (I/O2)
- net USB_DP: now also U4.6 (I/O1)
- net VUSB: now also C102.1, U4.5 (VBUS); no longer C4.1, U3.3 (VI)
- net at R4.2: now also U5.27 (PB4), U8.3 (A)
- net at R4.1: now also U5.28 (PB5)
- net SWCLK renamed SCLK
- net SCLK: now also U5.24 (PA14); no longer U105.1 (A)
- new net: U5.26 (PB3), U7.3 (A)
- new net: R104.1, U5.20 (PA10)
- new net: U5.25 (PA15), U8.5 (DIR)
- new net: R106.1, U8.4 (B)
- new net DM: U4.3 (I/O2), U5.21 (PA11)
- new net DP: U4.1 (I/O1), U5.22 (PA12)
- new net boot0: R105.2, U105.1 (A), U5.31 (BOOT0)
- new net en1.8v: U5.7 (PA1)
- no-connect marks 18 -> 17
Other:
- note added: "Add a resistor between PA1 and Tag Mirror"
- note removed: "DFU - pullup, weak pulldown on pin"
- note removed: "No need for pulldown on PA14 -- weak internal pull-down activated on reset"
- moved on the sheet: D1, J1, R1, R2, R3, SW1, SW2, U2

Commit message: added smps breakout board
Parts:
- removed D1: D_Schottky_Small, Diode_SMD:D_SOD-323, symbol Device:D_Schottky_Small
- added C6: 0.1uF, Capacitor_SMD:C_0402_1005Metric, symbol Device:C
- added R5: 1M, Resistor_SMD:R_0402_1005Metric, symbol Device:R
- added U6: TLV9001IDCKR, Package_TO_SOT_SMD:SOT-353_SC-70-5, symbol Amplifier_Operational:TLV9001IDCK
Connections:
- net TAG_VBAT is gone; now on net TAG_3V3: J101.6 (Pin_6), SW2.2 (B)
- net en1.8v is gone; now on net CSO: U5.7 (PA1)
- net +3V3: now also C6.1, U6.5 (V+); no longer U7.5 (DIR)
- net CSO: no longer U5.6 (PA0)
- net GND: now also C6.2, U6.2 (V-)
- net TAG_3V3: now also R5.2
- net at SW1.2 (B): now also SW2.1 (A)
- net TAG_SCK_EN: now reaches U5.30 (PB7)
- net TAG_SCK_EN: now also U7.5 (DIR)
- new net: R5.1, U6.1 (+)
- new net TAG_3V3_Valid: U5.6 (PA0), U6.3 (-), U6.4
- no-connect marks 17 -> 15
Other:
- note added: "Switch to 1.85v"
- moved on the sheet: C2, SW1, SW2

Commit message: checkpoint
Parts:
- removed U3: XC6206P182MR, Package_TO_SOT_SMD:SOT-23-3, symbol Regulator_Linear:XC6206PxxxMR
- added U3: AP2112K-1.8, Package_TO_SOT_SMD:SOT-23-5, symbol Regulator_Linear:AP2112K-1.8
Connections:
- net +1V8: now also U3.5 (VOUT)
- net +3V3: now also U7.5 (DIR), U3.1 (VIN)
- net GND: now also U3.2 (GND)
- net en1.8v: now reaches U5.29 (PB6)
- net en1.8v: now also U3.3 (EN)
- net TAG_SCK_EN: no longer names the net of U5.30 (PB7)
- net TAG_SCK_EN: no longer U7.5 (DIR)
Other:
- note added: "5 Pin package but pin 4 is defined as NC in datasheet"
- note removed: "Add a resistor between PA1 and Tag Mirror"
- note removed: "Switch to 1.85v"
