File: BoardDesigns/tagbase-lipo-v1/tagbase-lipo-v1.kicad_pcb (KiCad board)
At the start: 4 copper layers, 50.8 x 69.9 mm, 42 parts, among them J1 Conn_01x04_Female, J101 Conn_02x03_Odd_Even, J102 Conn_02x05_Odd_Even, J104 USB_B_Mini, J5 Conn_01x02, SW1 SW_SPDT, SW2 SW_SPDT, U1 XC6206P332MR, U105 Tactile Switch, U2 XC6808ANC28R-G, U3 AP2112K-1.8, U4 USBLC6-2P6, U5 STM32L432KBU6, U6 TLV9001IDCKR, U7 SN74LVC1T45DCK, U8 SN74LVC1T45DCK

Commit message: tagbase-lipo-v1: design review -- charger variant, charger caps, first config
Adds tagbase-lipo-v1-design-review.md and the board's first .kicad-happy.json,
and commits the changes the review produced plus the verified fab package.

Board changes:

- U2 changed from XC6808ANC28R-G to XC6808A4C28R-G. The two differ in exactly
  one field of the Torex part number -- the battery temperature monitor, N (none)
  vs 4 (JEITA). Charge voltage 4.20 V, 10 h hold, trickle enabled, 1 kHz abnormal
  status and USP-6B07 package are identical. On the xN, pin 5 is NF and the
  datasheet requires it OPEN, which made R2 wrong; on the A4 it is THIN and
  R2 = 10 kohm is the correct termination. The A4 is also less than half the
  price ($1.237 vs $2.7275).
- C9 (1 uF) added on /BAT, 1.56 mm from U2 pin 1, and C10 (1 uF) on VUSB,
  2.15 mm from U2 pin 6. These are the CL and CIN the datasheet's typical
  application circuit mandates; /BAT previously had no capacitor at all and the
  nearest cap to VIN was a 0.1 uF at 12.81 mm.
- The BOM's LCSC number for U2 no longer disagrees with its MPN. An export-tool
  mode had been auto-selecting LCSC numbers and picked C3682502 against a
  schematic MPN of XC6808ANC28R-G; that mode is off and MPN and part number now
  agree on the A4.
- LED note amended to record that 220 ohm is deliberate and 100 ohm measured too
  bright, so R102 no longer reads as an error.

Three findings in the review were raised in error and are recorded as withdrawn
rather than deleted, because each names a check that looked conclusive:

- The J101 NPTH holes sit 0.2032 mm apart, below the project's own rule. This is
  Mill-Max geometry, not a defect: J101 is a 855-22-0XX-10-001101 spring-loaded
  connector whose locating pegs are 1.04 mm on the connector's 1.27 mm row pitch.
  Verified against Mill-Max's own drawings -- signal hole 0.56 +/-0.08 (board
  0.610), pad 0.81 suggested (board 0.940), pitch and row spacing 1.27 exact.
  I had checked the footprint NAME rather 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
Parts:
- added C10: 1uF, Capacitor_SMD:C_0402_1005Metric, F.Cu at (137.1, 63.8)
- added C9: 1uF, Capacitor_SMD:C_0402_1005Metric, F.Cu at (135.5, 64.3)
- added R107: 2.2K, Resistor_SMD:R_0402_1005Metric, F.Cu at (134.3, 68.3)
- U2: value XC6808ANC28R-G -> XC6808A4C28R-G
Connections:
- U6 pad 3: /TAG_3V3_Valid -> Net-(U6--)
- U6 pad 4: /TAG_3V3_Valid -> Net-(U6--)
Routing:
- net /TAG_3V3_Valid: track 13.3 -> 5.45 mm
- net Net-(U6--): track 0.00 -> 6.78 mm
- net /BAT: track 13.9 -> 15.6 mm
- net GND: track 32.5 -> 34.1 mm, vias 27 -> 29
- net VUSB: track 52.2 -> 53.4 mm
