File: BoardDesigns/Archive/imutag-nand-bmp581/imutag-nand-bmp581.kicad_sch (KiCad schematic)
At the start: 37 parts, among them J201 CONN_02X04, J301 Conn_01x01, J302 Conn_01x01, J303 Conn_01x01, J304 Conn_01x01, J401 CONN_01X02, Q501 PMBT2222AMBYL, U1 TPS22916BYFPR, U2 BMM350, U3 BMP581, U302 stm32U375, U4 TPS7A02185PDQNR, U5 LSM6DSV16X, U501 RV-3028-C8, U6 GD5F1GQ5REYIGR

Commit message: ran design review on imutag-smps
Parts:
- removed U5: LSM6DSV16X, libraries:LGA14-L_2P59X3P1X0P5_STM, symbol lsm6dsv:LSM6DSV
- added U5: LSM6DSV, libraries:LGA14-L_2P59X3P1X0P5_STM, symbol libraries:LSM6DSV
- U6: value GD5F1GQ5REYIGR -> GD5F2GM7REYIGR; LCSC C2927042 -> C23706308; MPN GD5F1GQ5REYIGR -> GD5F2GM7REYIGR
Connections:
- net +1V8: now also U5.5 (VDD_IO), U5.8 (VDD)
- net AT25_MISO: now also U5.1 (SDO/SA0)
- net AT25_MOSI: now also U5.14 (SDA)
- net AT25_SCK: now also U5.13 (SCL)
- net GND: now also U5.2 (SDX), U5.3 (SCX), U5.6 (GND), U5.7 (GND)
- net LSM_CS: now also U5.12 (CS)
- net LSM_TRG: now also U5.9 (INT2)
- net WKUP1: now also U5.4 (INT1)
