File: BoardDesigns/imutag-nand-bmp581/imutag-nand-bmp581.kicad_pcb (KiCad board)
At the start: 4 copper layers, 21.5 x 11.5 mm, 37 parts, among them J201 CONN_02X04, J301 Conn_01x01, J302 Conn_01x01, J303 Conn_01x01, J304 Conn_01x01, J401 CONN_01X02, Q501 PMBT2222AMBYL, U1 TPS22916BYFPR, U2 BMM350, U3 BMP581, U302 stm32U375, U4 TPS7A02185PDQNR, U5 LSM6DSV16X, U501 RV-3028-C8, U6 GD5F1GQ5REYIGR

Commit message: added design review
Parts:
- removed D401: D, Diode_SMD:D_SOD-923
- U5: value LSM6DSV16X -> LSM6DSV
- U6: value GD5F1GQ5REYIGR -> GD5F2GM7REYIGR
Connections:
- C7 pad 1: VIN -> VBAT
- J201 pad 1: VIN -> VBAT
- U4 pad 3: VIN -> VBAT
- U4 pad 4: VIN -> VBAT
Routing:
- net VIN: track 20.2 -> 0.00 mm, vias 2 -> 0
- net VBAT: track 28.9 -> 27.3 mm
