File: BoardDesigns/imutag-nand-bmp581/imutag-nand-bmp581.kicad_sch (KiCad schematic)
At the start: 37 parts, among them J201 CONN_02X04, J301 Conn_01x01, J302 Conn_01x01, J303 Conn_01x01, J304 Conn_01x01, J401 CONN_01X02, Q501 PMBT2222AMBYL, U1 TPS22916BYFPR, U2 BMM350, U3 BMP581, U302 stm32U375, U4 TPS7A02185PDQNR, U5 LSM6DSV, U501 RV-3028-C8, U6 GD5F2GM7REYIGR

Commit message: added design review
Parts:
- removed D401: D, Diode_SMD:D_SOD-923, symbol Device:D_Schottky
- U1: MANUFACTURER (none) -> Texas Instruments
Connections:
- net VIN is gone; now on net VBAT: C7.1, J201.1 (Pin_1), U4.3 (EN), U4.4 (IN)
Other:
- note removed: "NEED TO LOOK AT POWER Do we need both vin and vbat? What is that diode for?"
Changed lines of the file:
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@@
 		)
 	)
-	(text "NEED TO LOOK AT POWER\nDo we need both vin and vbat?  \nWhat is that diode for?"
-		(exclude_from_sim no)
-		(at 172.72 45.212 0)
-		(effects
-			(font
-				(size 1.524 1.524)
-				(color 255 40 67 1)
-			)
-		)
-	)
 	(text "Tag Holes"
 		(exclude_from_sim no)
@@
 	)
 	(junction
-		(at 215.9 24.13)
+		(at 248.92 36.83)
 		(diameter 0)
 		(color 0 0 0 0)
 	)
 	(junction
-		(at 248.92 36.83)
+		(at 227.33 24.13)
 		(diameter 0)
 		(color 0 0 0 0)
 	)
 	(junction
-		(at 227.33 24.13)
+		(at 215.9 24.13)
 		(diameter 0)
 		(color 0 0 0 0)
@@
 	)
 	(junction
-		(at 215.9 31.75)
-		(diameter 0)
-		(color 0 0 0 0)
-	)
-	(junction
 		(at 25.4 148.59)
 		(diameter 0)
@@
 	)
 	(junction
+		(at 215.9 31.75)
+		(diameter 0)
+		(color 0 0 0 0)
+	)
+	(junction
 		(at 21.59 146.05)
 		(diameter 0)
@@
 	(wire
 		(pts
+			(xy 215.9 24.13) (xy 222.25 24.13)
+		)
+		(stroke
+			(width 0)
+			(type default)
+		)
+	)
+	(wire
+		(pts
 			(xy 19.05 148.59) (xy 25.4 148.59)
 		)
@@
 	(wire
 		(pts
+			(xy 215.9 24.13) (xy 215.9 31.75)
+		)
+		(stroke
+			(width 0)
+			(type default)
+		)
+	)
+	(wire
+		(pts
 			(xy 63.5 48.26) (xy 63.5 49.53)
 		)
@@
 	(wire
 		(pts
-			(xy 215.9 24.13) (xy 222.25 24.13)
-		)
-		(stroke
-			(width 0)
-			(type default)
-		)
-	)
-	(wire
-		(pts
 			(xy 240.03 59.69) (xy 240.03 67.31)
 		)
@@
 	)
 	(symbol
-		(lib_id "Device:D_Schottky")
-		(at 215.9 27.94 270)
-		(unit 1)
-		(body_style 1)
-		(exclude_from_sim no)
-		(in_bom yes)
-		(on_board yes)
-		(in_pos_files yes)
-		(dnp no)
-		(property "Reference" "D401"
-			(at 210.4136 27.94 0)
-			(show_name no)
-			(do_not_autoplace no)
-			(effects
-				(font
-					(size 1.27 1.27)
-				)
-			)
-		)
-		(property "Value" "D"
-			(at 212.725 27.94 0)
-			(show_name no)
-			(do_not_autoplace no)
-			(effects
-				(font
-					(size 1.27 1.27)
-				)
-			)
-		)
-		(property "Footprint" "Diode_SMD:D_SOD-923"
-			(at 215.9 27.94 0)
-			(hide yes)
-			(show_name no)
-			(do_not_autoplace no)
-			(effects
-				(font
-					(size 1.27 1.27)
-				)
-			)
-		)
-		(property "Datasheet" ""
-			(at 215.9 27.94 0)
-			(hide yes)
-			(show_name no)
-			(do_not_autoplace no)
-			(effects
-				(font
-					(size 1.27 1.27)
-				)
-			)
-		)
-		(property "Description" ""
-			(at 215.9 27.94 0)
-			(hide yes)
-			(show_name no)
-			(do_not_autoplace no)
-			(effects
-				(font
-					(size 1.27 1.27)
-				)
-			)
-		)
-		(property "MFN" "COMCHIP"
-			(at 215.9 27.94 0)
-			(hide yes)
-			(show_name no)
-			(do_not_autoplace no)
-			(effects
-				(font
-					(size 1.27 1.27)
-				)
-			)
-		)
-		(property "MPN" "CDBQC0130L-HF"
-			(at 215.9 27.94 0)
-			(hide yes)
-			(show_name no)
-			(do_not_autoplace no)
-			(effects
-				(font
-					(size 1.27 1.27)
-				)
-			)
-		)
-		(property "LCSC" "C2886012"
-			(at 215.9 27.94 0)
-			(hide yes)
-			(show_name no)
-			(do_not_autoplace no)
-			(effects
-				(font
-					(size 1.524 1.524)
-				)
-			)
-		)
-		(pin "1"
-		)
-		(pin "2"
-		)
-		(instances
-			(project "imutag-nand-bmp581"
-				(path "/e44ca67a-43be-444b-8652-f54825a2eb6f"
-					(reference "D401")
-					(unit 1)
-				)
-			)
-		)
-	)
-	(symbol
 		(lib_id "BitTagNG:RV-3028-C7-AccelTag")
 		(at 223.52 63.5 0)
@@
 	)
 	(symbol
-		(lib_id "power:PWR_FLAG")
-		(at 104.14 21.59 0)
-		(unit 1)
-		(body_style 1)
-		(exclude_from_sim no)
-		(in_bom yes)
-		(on_board yes)
-		(in_pos_files yes)
-		(dnp no)
-		(fields_autoplaced yes)
-		(property "Reference" "#FLG01"
-			(at 104.14 19.685 0)
-			(hide yes)
-			(show_name no)
-			(do_not_autoplace no)
-			(effects
-				(font
-					(size 1.27 1.27)
-				)
-			)
-		)
-		(property "Value" "PWR_FLAG"
-			(at 104.14 16.51 0)
-			(show_name no)
-			(do_not_autoplace no)
-			(effects
-				(font
-					(size 1.27 1.27)
-				)
-			)
-		)
-		(property "Footprint" ""
-			(at 104.14 21.59 0)
-			(hide yes)
-			(show_name no)
-			(do_not_autoplace no)
-			(effects
-				(font
-					(size 1.27 1.27)
-				)
-			)
-		)
-		(property "Datasheet" ""
-			(at 104.14 21.59 0)
-			(hide yes)
-			(show_name no)
-			(do_not_autoplace no)
-			(effects
-				(font
-					(size 1.27 1.27)
-				)
-			)
-		)
-		(property "Description" "Special symbol for telling ERC where power comes from"
-			(at 104.14 21.59 0)
-			(hide yes)
-			(show_name no)
-			(do_not_autoplace no)
-			(effects
-				(font
-					(size 1.27 1.27)
-				)
-			)
-		)
-		(pin "1"
-		)
-		(instances
-			(project "imutag-nand-bmp581"
-				(path "/e44ca67a-43be-444b-8652-f54825a2eb6f"
-					(reference "#FLG01")
-					(unit 1)
-				)
-			)
-		)
-	)
-	(symbol
 		(lib_id "Device:C")
 		(at 248.92 29.21 0)
@@
 			)
 		)
+		(property "MANUFACTURER" "Texas Instruments"
+			(at 46.99 43.18 0)
+			(hide yes)
+			(show_name no)
+			(do_not_autoplace no)
+			(effects
+				(font
+					(size 1.27 1.27)
+				)
+				(justify bottom)
+			)
+		)
