File: BoardDesigns/imutag-nand-bmp581/imutag-nand-bmp581.kicad_sch (KiCad schematic)
At the start: 36 parts, among them J201 CONN_02X04, J301 Conn_01x01, J302 Conn_01x01, J303 Conn_01x01, J304 Conn_01x01, J401 CONN_01X02, Q501 PMBT2222AMBYL, U1 TPS22916BYFPR, U2 BMM350, U3 BMP581, U302 stm32U375, U4 TPS7A02185PDQNR, U5 LSM6DSV, U501 RV-3028-C8, U6 GD5F2GM7REYIGR

Commit message: imutag-nand-bmp581: fab-ready for PCBWay, plus stale-project cleanup
Design review round 2, covering the PCBWay fabrication package that did not
exist at the 2026-08-26 review. Closed ready to fabricate.

Board fixes
- Inner planes were flush with the routed profile: In1.Cu (+1V8) and In2.Cu
  (GND) both sat 0.0005 mm from the edge, separated by 0.08 mm of core, with a
  credible burr path from the regulated rail to ground. Invisible to DRC because
  min_copper_edge_clearance was 0. Now 0.3005 mm, rule set to 0.3 and enforced.
- Via annular ring raised 0.1016 -> 0.1524 mm (4.00 -> 6.00 mil) on all 44 vias
  to meet PCBWay's published minimum: pad 0.5048 / drill 0.20, now a single
  drill tool. Shrinking the drill is what buys the ring here; pad growth fails
  against the zones' 0.508 mm connect_pads clearance.
- C4 re-sourced to GRM155Z71A225KE01D (2.2 uF 10 V X7R 0402, LCSC C2997286).
  Bosch's recommended TDK CGB4B3X7R0J225K055AB is obsolete and is an 0805, so it
  was never a drop-in for the 0402 land.
- RV-3028-C8 footprint silk raised to 0.15 mm.

Verified: DRC 0 violations / 0 unconnected / 0 parity; ERC 1 accepted VBAT/VIN
warning; PTH 44 = via count, NPTH 4 = J301-J304; 15 BOM lines / 30 placements
matching the CPL exactly, every line with MPN and LCSC. The 10-01-52 export is
confirmed to match the board on disk.

Production package
- Only the final export, 2026-09-01-10-01-52, is kept; six superseded ones are
  pruned.
- Its gerber archive is committed with `git add -f`, overriding the repo-wide
  *.zip rule in BoardDesigns/.gitignore. Without that the commit would carry
  only the BOM, CPL and netlist, and the package actually sent to the fab would
  not be reproducible: plugin output is not byte-identical to a kicad-cli
  re-plot, so the board file alone does not pin it down. 46 kB.

Stale BitTagNG project files removed repo-wide
- analysis/2026-08-26_1027-2/pcb.json recorded rules_source as
  BitTagNG-LIS2DU12.kicad_pcb-back.kicad_pro, so every rule-deri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
Parts:
- C4: LCSC C237392 -> C2997286; MPN GRM155R6YA225KE11D -> GRM155Z71A225KE01D
- U501: value RV-3028-C8 -> RV-3028-C8-32.768kHz-1PPM-TA-QC; symbol BitTagNG:RV-3028-C7-AccelTag -> libraries:RV-3028-C7
Changed lines of the file:
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@@
 	(wire
 		(pts
+			(xy 241.3 115.57) (xy 243.84 115.57)
+		)
+		(stroke
+			(width 0)
+			(type default)
+		)
+	)
+	(wire
+		(pts
 			(xy 46.99 97.79) (xy 46.99 102.87)
 		)
@@
 	)
 	(symbol
-		(lib_id "BitTagNG:RV-3028-C7-AccelTag")
+		(lib_id "libraries:RV-3028-C7")
 		(at 223.52 63.5 0)
 		(unit 1)
@@
 			)
 		)
-		(property "Value" "RV-3028-C8"
+		(property "Value" "RV-3028-C8-32.768kHz-1PPM-TA-QC"
 			(at 223.52 56.1086 0)
 			(show_name no)
@@
 			)
 		)
-		(property "LCSC" "C237392"
+		(property "LCSC" "C2997286"
 			(at 85.09 156.21 0)
 			(hide yes)
@@
 			)
 		)
-		(property "MPN" "GRM155R6YA225KE11D"
+		(property "MPN" "GRM155Z71A225KE01D"
 			(at 85.09 156.21 0)
 			(hide yes)
@@
 					(unit 1)
 				)
+			)
+		)
+	)
+	(symbol
+		(lib_id "power:PWR_FLAG")
+		(at 241.3 115.57 0)
+		(unit 1)
+		(body_style 1)
+		(exclude_from_sim no)
+		(in_bom yes)
+		(on_board yes)
+		(in_pos_files yes)
+		(dnp no)
+		(property "Reference" "#FLG0103"
+			(at 241.3 113.665 0)
+			(hide yes)
+			(show_name no)
+			(do_not_autoplace no)
+			(effects
+				(font
+					(size 1.27 1.27)
+				)
+			)
+		)
+		(property "Value" "PWR_FLAG"
+			(at 241.3 111.76 0)
+			(show_name no)
+			(do_not_autoplace no)
+			(effects
+				(font
+					(size 1.27 1.27)
+				)
+			)
+		)
+		(property "Footprint" ""
+			(at 241.3 115.57 0)
+			(hide yes)
+			(show_name no)
+			(do_not_autoplace no)
+			(effects
+				(font
+					(size 1.27 1.27)
+				)
+			)
+		)
+		(property "Datasheet" ""
+			(at 241.3 115.57 0)
+			(hide yes)
+			(show_name no)
+			(do_not_autoplace no)
+			(effects
+				(font
+					(size 1.27 1.27)
+				)
+			)
+		)
+		(property "Description" "Special symbol for telling ERC where power comes from"
+			(at 241.3 115.57 0)
+			(hide yes)
+			(show_name no)
+			(do_not_autoplace no)
+			(effects
+				(font
+					(size 1.27 1.27)
+				)
+			)
+		)
+		(pin "1"
+		)
+		(instances
+			(project "imutag-nand-bmp581"
+				(path "/e44ca67a-43be-444b-8652-f54825a2eb6f"
+					(reference "#FLG0103")
+					(unit 1)
+				)
