File: BoardDesigns/imutag-smps/imutag-smps.kicad_sch (KiCad schematic)
At the start: 36 parts, among them J201 CONN_02X04, J301 Conn_01x01, J302 Conn_01x01, J303 Conn_01x01, J304 Conn_01x01, J401 CONN_01X02, Q501 PMBT2222AMBYL, U1 TPS22916BYFPR, U2 BMM350, U3 BMP581, U302 stm32U375, U4 TPS62840YBGR, U5 LSM6DSV16X, U501 RV-3028-C8, U6 GD5F2GM7REYIGR

Commit message: ran design review on imutag-smps
Parts:
- removed U5: LSM6DSV16X, libraries:LGA14-L_2P59X3P1X0P5_STM, symbol lsm6dsv:LSM6DSV
- added U5: LSM6DSV, libraries:LGA14-L_2P59X3P1X0P5_STM, symbol libraries:LSM6DSV
Connections:
- net +1V8: now also U5.5 (VDD_IO), U5.8 (VDD)
- net AT25_MISO: now also U5.1 (SDO/SA0)
- net AT25_MOSI: now also U5.14 (SDA)
- net AT25_SCK: now also U5.13 (SCL)
- net GND: now also U5.2 (SDX), U5.3 (SCX), U5.6 (GND), U5.7 (GND)
- net LSM_CS: now also U5.12 (CS)
- net LSM_TRG: now also U5.9 (INT2)
- net WKUP1: now also U5.4 (INT1)
Changed lines of the file:
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@@
+	)
+	(symbol
+		(lib_id "libraries:LSM6DSV")
+		(at 191.77 138.43 0)
+		(unit 1)
+		(body_style 1)
+		(exclude_from_sim no)
+		(in_bom yes)
+		(on_board yes)
+		(in_pos_files yes)
+		(dnp no)
+		(fields_autoplaced yes)
+		(property "Reference" "U5"
+			(at 217.17 128.27 0)
+			(show_name no)
+			(do_not_autoplace no)
+			(effects
+				(font
+					(size 1.524 1.524)
+				)
+			)
+		)
+		(property "Value" "LSM6DSV"
+			(at 217.17 130.81 0)
+			(show_name no)
+			(do_not_autoplace no)
+			(effects
+				(font
+					(size 1.524 1.524)
+				)
+			)
+		)
+		(property "Footprint" "libraries:LGA14-L_2P59X3P1X0P5_STM"
+			(at 192.532 134.112 0)
+			(hide yes)
+			(show_name no)
+			(do_not_autoplace no)
+			(effects
+				(font
+					(size 1.27 1.27)
+					(italic yes)
+				)
+			)
+		)
+		(property "Datasheet" "LSM6DSV"
+			(at 185.166 136.398 0)
+			(hide yes)
+			(show_name no)
+			(do_not_autoplace no)
+			(effects
+				(font
+					(size 1.27 1.27)
+					(italic yes)
+				)
+			)
+		)
+		(property "Description" ""
+			(at 191.77 138.43 0)
+			(hide yes)
+			(show_name no)
+			(do_not_autoplace no)
+			(effects
+				(font
+					(size 1.27 1.27)
+				)
+			)
+		)
+		(property "LCSC" "C5267399"
+			(at 191.77 138.43 0)
+			(hide yes)
+			(show_name no)
+			(do_not_autoplace no)
+			(effects
+				(font
+					(size 1.27 1.27)
+				)
+			)
+		)
+		(property "MFN" "STM microelectronics"
+			(at 191.77 138.43 0)
+			(hide yes)
+			(show_name no)
+			(do_not_autoplace no)
+			(effects
+				(font
+					(size 1.27 1.27)
+				)
+			)
+		)
+		(property "MPN" "LSM6DSV"
+			(at 191.77 138.43 0)
+			(hide yes)
+			(show_name no)
+			(do_not_autoplace no)
+			(effects
+				(font
+					(size 1.27 1.27)
+				)
+			)
+		)
+		(pin "14"
+		)
+		(pin "8"
+		)
+		(pin "3"
+		)
+		(pin "2"
+		)
+		(pin "7"
+		)
+		(pin "9"
+		)
+		(pin "6"
+		)
+		(pin "4"
+		)
+		(pin "5"
+		)
+		(pin "10"
+		)
+		(pin "13"
+		)
+		(pin "12"
+		)
+		(pin "11"
+		)
+		(pin "1"
+		)
+		(instances
+			(project "imutag-smps"
+				(path "/e44ca67a-43be-444b-8652-f54825a2eb6f"
+					(reference "U5")
+					(unit 1)
+				)
+			)
+		)
 	)
 	(symbol
@@
 					(unit 1)
 				)
-			)
-		)
-	)
-	(symbol
-		(lib_id "lsm6dsv:LSM6DSV")
-		(at 191.77 138.43 0)
-		(unit 1)
-		(body_style 1)
-		(exclude_from_sim no)
-		(in_bom yes)
-		(on_board yes)
-		(in_pos_files yes)
-		(dnp no)
-		(fields_autoplaced yes)
-		(property "Reference" "U5"
-			(at 217.17 128.27 0)
-			(show_name no)
-			(do_not_autoplace no)
-			(effects
-				(font
-					(size 1.524 1.524)
-				)
-			)
-		)
-		(property "Value" "LSM6DSV16X"
-			(at 217.17 130.81 0)
-			(show_name no)
-			(do_not_autoplace no)
-			(effects
-				(font
-					(size 1.524 1.524)
-				)
-			)
-		)
-		(property "Footprint" "libraries:LGA14-L_2P59X3P1X0P5_STM"
-			(at 191.77 138.43 0)
-			(hide yes)
-			(show_name no)
-			(do_not_autoplace no)
-			(effects
-				(font
-					(size 1.27 1.27)
-					(italic yes)
-				)
-			)
-		)
-		(property "Datasheet" "LSM6DSV16X"
-			(at 191.77 138.43 0)
-			(hide yes)
-			(show_name no)
-			(do_not_autoplace no)
-			(effects
-				(font
-					(size 1.27 1.27)
-					(italic yes)
-				)
-			)
-		)
-		(property "Description" ""
-			(at 191.77 138.43 0)
-			(hide yes)
-			(show_name no)
-			(do_not_autoplace no)
-			(effects
-				(font
-					(size 1.27 1.27)
-				)
-			)
-		)
-		(property "MFN" "STMicroelectronics"
-			(at 191.77 138.43 0)
-			(hide yes)
-			(show_name no)
-			(do_not_autoplace no)
-			(effects
-				(font
-					(size 1.524 1.524)
-				)
-			)
-		)
-		(property "MPN" "LSM6DSV16XTR"
-			(at 191.77 138.43 0)
-			(hide yes)
-			(show_name no)
-			(do_not_autoplace no)
-			(effects
-				(font
-					(size 1.524 1.524)
-				)
-			)
-		)
-		(property "LCSC" "C5267406"
-			(at 191.77 138.43 0)
-			(hide yes)
-			(show_name no)
-			(do_not_autoplace no)
-			(effects
-				(font
-					(size 1.524 1.524)
-				)
-			)
-		)
-		(pin "14"
-		)
-		(pin "8"
-		)
-		(pin "3"
-		)
-		(pin "2"
-		)
-		(pin "7"
-		)
-		(pin "9"
-		)
-		(pin "6"
-		)
-		(pin "4"
-		)
-		(pin "5"
-		)
-		(pin "10"
-		)
-		(pin "13"
-		)
-		(pin "12"
-		)
-		(pin "11"
-		)
-		(pin "1"
-		)
-		(instances
-			(project "imutag-smps"
-				(path "/e44ca67a-43be-444b-8652-f54825a2eb6f"
-					(reference "U5")
-					(unit 1)
-				)

Commit message: added design review
Other:
- note removed: "NEED TO LOOK AT POWER Do we need both vin and vbat? What is that diode for?"
- note removed: "NEED TO SWITCH TO 2GB"
Changed lines of the file:
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@@
-		)
-	)
-	(text "NEED TO LOOK AT POWER\nDo we need both vin and vbat?  \nWhat is that diode for?"
-		(exclude_from_sim no)
-		(at 169.926 65.532 0)
-		(effects
-			(font
-				(size 1.524 1.524)
-				(color 255 40 67 1)
-			)
 		)
 	)
@@
 		)
 	)
-	(text "NEED TO SWITCH TO 2GB"
-		(exclude_from_sim no)
-		(at 34.036 61.468 0)
-		(effects
-			(font
-				(size 1.524 1.524)
-				(color 255 51 22 1)
-			)
-		)
-	)
