File: BoardDesigns/imutag-smps/imutag-smps.kicad_sch (KiCad schematic)
At the start: 36 parts, among them J201 CONN_02X04, J301 Conn_01x01, J302 Conn_01x01, J303 Conn_01x01, J304 Conn_01x01, J401 CONN_01X02, Q501 PMBT2222AMBYL, U1 TPS22916BYFPR, U2 BMM350, U3 BMP581, U302 stm32U375, U4 TPS62840YBGR, U5 LSM6DSV, U501 RV-3028-C8, U6 GD5F2GM7REYIGR

Commit message: imutag-smps: design review 2 — switching converter, magnetics, pin map
Review of the SMPS power stage and the current board state, following 2026-08-26.
NOT ordered: one architectural question is still open.

Board changes
- L1 reroute: /AT25_MOSI on B.Cu moved 1.13 -> 1.38 mm from the inductor centre,
  now clear of the 1.6 x 2.0 mm body outline; /AT25_SCK 1.57 -> 1.69 mm.
- BMP581 symbol updated from the library: VSS pins 3/8/9 were typed power_out where
  libraries:BMP581 has power_in. That silently drove the GND net; correcting it
  exposed power_pin_not_driven on U1 pin B1 - the same latent bug as
  RV-3028-C7-AccelTag on imutag-nand-bmp581. Fixed with a PWR_FLAG (#FLG02) on GND.
- #FLG01 moved from /Flash 1V8, which U1's VOUT already drives, to +1V8, which the
  TPS62840 symbol leaves undriven because VOS is correctly typed as a sense input.
  That cleared both remaining ERC errors.
- Edge clearance and annular ring brought in line with the sibling: inner copper
  0.3005 mm from the profile, all 47 vias at 0.1524 mm (6.00 mil), single drill.

Verified: DRC 0 violations / 0 unconnected / 0 parity. ERC 0 violations, and 0
errors with all 24 exclusions cleared. Export 2026-09-02-08-29-52 matches the board
- 300/300 fill vertices on both inner planes, 412/412 track starts, PTH 47 = 47
vias, NPTH 4. Superseded exports pruned; the gerber archive is force-added past the
repo-wide *.zip rule so the package is recoverable from the commit.

Findings
1. The TPS62840YBG has NO MODE pin - datasheet 8.3.3, "not available in the YBG
   package". Forced PWM is unavailable, so at 1-2.2 mA the converter sits in PFM
   and switching noise is bursty, load-dependent and not selectable. This removes
   the option the family-level SMPS-vs-LDO decision rested on: the buck keeps its
   full ~1.85x battery-life advantage precisely because the mode that would have
   erased it cannot be chosen. Not a defect - a decision to make deliberately.
2. Switching-loop layout reviewed, the item R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
Parts:
- C10, C11, C12, C4, C504, C505, C506, C507, C6, C7, C8, R2, R3: KiLib_Generator (none) -> SMD_2terminal_chip_molded
- U302, U6: KiLib_Generator (none) -> package/no_lead
- U501: symbol BitTagNG:RV-3028-C7-AccelTag -> tag_library:RV-3028-C7

Commit message: imutag-smps: pin alternates, tighter DRC, symbol hygiene; prune to current outputs
Continues the 2026-09-02 review. Still NOT ordered - finding 1 (the TPS62840YBG has
no MODE pin, so the converter is PFM-only) remains the open architectural question.

Design
- All 12 U302 pin alternates declared on the schematic, so pin intent is stated by
  the design rather than inferred by the reviewer. PB4 is LPTIM1_CH2, not a GPIO;
  PC14 is RCC_OSC32_IN, feeding the LSE in bypass mode from the RV-3028's 32.768 kHz
  CLKOUT. LPTIM1 divides that onto PB4 to trigger the IMU in hardware while the CPU
  is stopped, at 1 PPM rather than internal-RC accuracy.
- RV-3028 CLKOUT retyped input -> output, in the library and the schematic cache.
  Correct direction and required for coherence with PC14 declaring RCC_OSC32_IN.
- BMP581 symbol updated from library; pin maps now identical, VSS pins power_in.
- U501 repointed tag_library:RV-3028-C7 -> libraries:RV-3028-C7. 'tag_library' is not
  in this project's sym-lib-table and resolved only through the user-level table, so
  the reference was machine-local and would fail on a fresh clone while ERC stayed
  quiet - the cached lib_symbols entry hides it. Connectivity verified unchanged:
  37 nets, 138 pin connections.
- DRC severities tightened: npth_inside_courtyard and pth_inside_courtyard
  ignore -> warning, track_not_centered_on_via ignore -> ERROR. The last matters
  because the board was moved to a 6.00 mil annular ring for margin, which an
  off-centre track endpoint would silently give back.

Verified: DRC 0 violations / 0 unconnected / 0 parity with the tightened rules. ERC
0 violations, and 0 errors with all 17 exclusions cleared. Promoting every remaining
'ignore' yields only 5 missing_courtyard hits, all on mounting holes and battery
lands. Export 2026-09-03-07-51-02 matches the board: 300/300 fill vertices on both
inner planes, 392/392 track starts, edge 0.3005 mm, PTH 44 = 44 vias, BOM 16 lines /
27 placements matching the CPL.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
Parts:
- removed C10: 1uf, Capacitor_SMD:C_0201_0603Metric, symbol Device:C
- removed C507: 0.1uf, Capacitor_SMD:C_0201_0603Metric, symbol Device:C
- removed U1: TPS22916BYFPR, libraries:IC_TPS22916BYFPR, symbol libraries:TPS22916BYFPR
- U501: symbol tag_library:RV-3028-C7 -> libraries:RV-3028-C7
Connections:
- net Flash 1V8 is gone; now on net +1V8: C11.1, C504.1, U6.3 (~{WP}/SIO2), U6.7 (~{HOLD}/SIO3), U6.8 (VCC)
- net FLASH_PWR: no longer names the net of U302.18 (PA8)
- no-connect marks 9 -> 10
Other:
- title: IMU Tag with NAND and BMM350 -> IMU Tag with NAND and BMM350 and SMPS
- moved on the sheet: C11, C504, U6
