File: BoardDesigns/BitPresTagBMP585/BitPresTagBMP585.kicad_sch (KiCad schematic)
At the start: 28 parts, among them J201 CONN_02X04, J301 Conn_01x01, J302 Conn_01x01, J303 Conn_01x01, J304 Conn_01x01, J401 CONN_01X02, Q501 PMBT2222AMBYL, U1 at25ex321D-UUN, U2 ADXL367BCCZ-RL7, U3 BMP585, U302 stm32l431kc, U501 RV-3028-C8-32.768kHz-1PPM-TA-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

Commit message: BitPresTagBMP585: settle U1, close the reset finding, add verified fab package
Replaces an earlier commit that was mislabelled and incomplete: it claimed
to cover only the reset network, but a blanket `git add -A` had also swept
in the U1 label change and three quarters of a production package. The
gerber archive was silently dropped because BoardDesigns/.gitignore
excludes *.zip -- the exact failure mode the working notes warn about, where
the BOM, CPL and netlist land in git but the thing actually sent to the fab
does not. The archive is force-added here (39 kB).

U1 settled on AT25FF321A-UUN-T; Value now matches MPN in both schematic and
PCB. The two candidates are pin-identical, so this was a BOM-consistency
choice rather than a board risk. One firmware consequence: the AT25FF321A
has no 256-byte page erase, so its smallest erase is a 4 kByte block. Small
in-place record rewrites now need a read-modify-write of a 4 kB block;
append-only logging with 4 kB-aligned erases is unaffected.

Q501's base series resistor lives on the external connecting board that
mates through J201 -- confirmed by the designer, same arrangement as
BitTagNG. mating_design now describes the board correctly (it is not
self-contained, as the copied-in config had claimed) and adds a
baseboard_contract block: supply a ~4.7-10 kOhm base resistor to J201.5,
and drive J201.5 HIGH to assert reset.

Production package pcbway_production/2026-09-04-19-11-58 verified against
the board by geometry rather than mtime:
  - 60/60 sampled F.Cu/B.Cu track endpoints present in the gerbers
  - 40/40 vias reconciled with the PTH drill at 0.2007 mm, every one
    measuring a 0.1524 mm annular ring
  - 4 NPTH at 1.0998 mm; outline exactly 18.0 x 10.0 mm
  - inner planes 17.399 x 9.399 mm, confirming the 0.3 mm edge clearance
  - all 11 gerbers plus both drill files present
  - BOM 22 designators == CPL 22 placements, both including C8 and R2
J201, J301-J304 and J401 are correctly absent from both: solder tagpoin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
Parts:
- U1: value at25ex321D-UUN -> 724-AT25FF321A-UUN-T
Changed lines of the file:
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@@
 			)
 		)
-		(property "Value" "at25ex321D-UUN"
+		(property "Value" "724-AT25FF321A-UUN-T"
 			(at 58.42 26.0604 0)
 			(show_name no)

Commit message: BitPresTagBMP585: close the review -- U302 label and LPS_VDD net name
U302 Value corrected stm32l431kc -> STM32L432KCU6, matching its MPN in both
schematic and PCB. Value now agrees with MPN on every part.

The switched sensor supply is labelled LPS_VDD. LPS_PWR now correctly names
only the PB1 -> R2 stub, and the PP-001 suppression is re-keyed from the
unnamed net __unnamed_13 to LPS_VDD, so it no longer breaks on the next
schematic edit. PP-001 remains suppressed: U3's supply comes from a GPIO
through a resistor by design, so it has no DC path to a rail.

Verified: KiCad DRC 0 violations / 0 unconnected, KiCad ERC 0 violations,
padnet_crosscheck 28 footprints / 0 mismatches.

The existing fab package predates both edits, so it should be regenerated
before ordering. The copper is unaffected -- all 305 outer-layer track
endpoints still match the board, 40 vias at 0.5048/0.2 mm, outline
18 x 10 mm -- and the BOM's MPN column is already correct. It is stale only
in the cosmetic BOM Value column and the netlist.ipc net labels.

Every finding this review raised is now closed.

Co-Authored-By: Claude Opus 5 (1M context) <noreply@anthropic.com>
Parts:
- U302: value stm32l431kc -> STM32L432KCU6
Connections:
- net LPS_VDD: now reaches C3.1, C5.1, R2.1, U3.4 (VDDIO), U3.8 (VDD)
Changed lines of the file:
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@@
+		)
+	)
+	(label "LPS_VDD"
+		(at 220.98 135.89 0)
+		(effects
+			(font
+				(size 1.524 1.524)
+			)
+			(justify left bottom)
 		)
 	)
@@
 			)
 		)
-		(property "Value" "stm32l431kc"
+		(property "Value" "STM32L432KCU6"
 			(at 128.27 93.98 0)
 			(show_name no)
