File: BoardDesigns/Tags/BitPresTagBMP585/BitPresTagBMP585.kicad_pcb (KiCad board)
At the start: 4 copper layers, 18 x 10 mm, 28 parts, among them J201 CONN_02X04, J301 Conn_01x01, J302 Conn_01x01, J303 Conn_01x01, J304 Conn_01x01, J401 CONN_01X02, Q501 PMBT2222AMBYL, U1 724-AT25FF321A-UUN-T, U2 ADXL367BCCZ-RL7, U3 BMP585, U302 STM32L432KCU6, U501 RV-3028-C8-32.768kHz-1PPM-TA-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

Commit message: update BitPresTagBMP585
Parts:
- U302: value STM32L432KCU6 -> STM32L432KCU6TR
Changed lines of the file:
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@@
 			(drillshape 0)
 			(scaleselection 1)
-			(outputdirectory "../../Mechanical/BitPresTag/")
+			(outputdirectory "../../../Mechanical/BitPresTag/")
 		)
 	)
@@
 			)
 		)
-		(attr through_hole exclude_from_pos_files exclude_from_bom)
+		(attr through_hole exclude_from_pos_files exclude_from_bom dnp)
 		(duplicate_pad_numbers_are_jumpers no)
 		(pad "" np_thru_hole circle
@@
 			)
 		)
-		(attr smd exclude_from_pos_files exclude_from_bom)
+		(attr smd exclude_from_pos_files exclude_from_bom dnp)
 		(duplicate_pad_numbers_are_jumpers no)
 		(fp_text user "-"
@@
 			)
 		)
-		(property "LCSC" "C181047"
+		(property "LCSC" "C408130"
 			(at 258.6628 -37.766 90)
 			(layer "F.Fab")
@@
 			)
 		)
-		(property "MPN" "GRM033C81E104KE14D"
+		(property "MPN" "GRM033R61A104ME15D"
 			(at 258.6628 -37.766 90)
 			(layer "F.Fab")
@@
 			)
 		)
-		(property "LCSC" "C181047"
+		(property "LCSC" "C408130"
 			(at 0 0 0)
 			(layer "F.Fab")
@@
 			)
 		)
-		(property "MPN" "GRM033C81E104KE14D"
+		(property "MPN" "GRM033R61A104ME15D"
 			(at 0 0 0)
 			(layer "F.Fab")
@@
 			)
 		)
-		(attr through_hole exclude_from_pos_files exclude_from_bom)
+		(attr through_hole exclude_from_pos_files exclude_from_bom dnp)
 		(duplicate_pad_numbers_are_jumpers no)
 		(pad "" np_thru_hole circle
@@
 			)
 		)
-		(attr through_hole exclude_from_pos_files exclude_from_bom)
+		(attr through_hole exclude_from_pos_files exclude_from_bom dnp)
 		(duplicate_pad_numbers_are_jumpers no)
 		(pad "" np_thru_hole circle
@@
 			)
 		)
-		(attr through_hole exclude_from_pos_files exclude_from_bom)
+		(attr through_hole exclude_from_pos_files exclude_from_bom dnp)
 		(duplicate_pad_numbers_are_jumpers no)
 		(pad "" np_thru_hole circle
@@
 			)
 		)
-		(property "MPN" "GRM033C81E104KE14D"
+		(property "MPN" "GRM033R61A104ME15D"
 			(at 0 0 270)
 			(unlocked yes)
@@
 			)
 		)
-		(property "LCSC" "C181047"
+		(property "LCSC" "C408130"
 			(at 0 0 270)
 			(unlocked yes)
@@
 			)
 		)
-		(property "MPN" "GRM033C81E104KE14D"
+		(property "MPN" "GRM033R61A104ME15D"
 			(at 0 0 270)
 			(unlocked yes)
@@
 			)
 		)
-		(property "LCSC" "C181047"
+		(property "LCSC" "C408130"
 			(at 0 0 270)
 			(unlocked yes)
@@
 			)
 		)
-		(property "MPN" "GRM033C81E104KE14D"
+		(property "MPN" "GRM033R61A104ME15D"
 			(at 0 0 270)
 			(unlocked yes)
@@
 			)
 		)
-		(property "LCSC" "C181047"
+		(property "LCSC" "C408130"
 			(at 0 0 270)
 			(unlocked yes)
@@
 			)
 		)
-		(attr smd exclude_from_pos_files exclude_from_bom)
+		(attr smd exclude_from_pos_files exclude_from_bom dnp)
 		(duplicate_pad_numbers_are_jumpers no)
 		(fp_line
@@
 			)
 		)
-		(property "LCSC" "C181047"
+		(property "LCSC" "C408130"
 			(at 0 0 90)
 			(layer "B.Fab")
@@
 			)
 		)
-		(property "MPN" "GRM033C81E104KE14D"
+		(property "MPN" "GRM033R61A104ME15D"
 			(at 0 0 90)
 			(layer "B.Fab")
@@
 			)
 		)
-		(property "Value" "STM32L432KCU6"
+		(property "Value" "STM32L432KCU6TR"
 			(at 0 -3.82 0)
 			(layer "B.Fab")
@@
 			)
 		)
-		(property "DISTPN" "497-16578-ND"
+		(property "DISTPN" "497-STM32L432KCU6TR-ND"
 			(at 0 0 0)
 			(layer "B.Fab")
@@
 			)
 		)
-		(property "MPN" "STM32L432KCU6"
+		(property "MPN" "STM32L432KCU6TR"
 			(at 0 0 0)
 			(layer "B.Fab")
@@
 			)
 		)
-		(property "LCSC" "C181047"
+		(property "LCSC" "C408130"
 			(at 284.34 -218.142 90)
 			(layer "B.Fab")
@@
 			)
 		)
-		(property "MPN" "GRM033C81E104KE14D"
+		(property "MPN" "GRM033R61A104ME15D"
 			(at 284.34 -218.142 90)
 			(layer "B.Fab")
@@
 			)
 		)
-		(property "MPN" "GRM033C81E104KE14D"
+		(property "MPN" "GRM033R61A104ME15D"
 			(at 0 0 180)
 			(unlocked yes)
@@
 			)
 		)
-		(property "LCSC" "C181047"
+		(property "LCSC" "C408130"
 			(at 0 0 0)
 			(unlocked yes)
@@
 			)
 		)
-		(property "MPN" "GRM033C81E104KE14D"
+		(property "MPN" "GRM033R61A104ME15D"
 			(at 0 0 180)
 			(unlocked yes)
@@
 			)
 		)
-		(property "LCSC" "C181047"
+		(property "LCSC" "C408130"
 			(at 0 0 0)
 			(unlocked yes)
