File: BoardDesigns/Tags/BitPresTagBMP585/BitPresTagBMP585.kicad_sch (KiCad schematic)
At the start: 28 parts, among them J201 CONN_02X04, J301 Conn_01x01, J302 Conn_01x01, J303 Conn_01x01, J304 Conn_01x01, J401 CONN_01X02, Q501 PMBT2222AMBYL, U1 724-AT25FF321A-UUN-T, U2 ADXL367BCCZ-RL7, U3 BMP585, U302 STM32L432KCU6, U501 RV-3028-C8-32.768kHz-1PPM-TA-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

Commit message: update BitPresTagBMP585
Parts:
- C1, C2, C3, C5, C501, C502, C503, C504, C7: LCSC C181047 -> C408130; MPN GRM033C81E104KE14D -> GRM033R61A104ME15D
- J201, J301, J302, J303, J304, J401: now not fitted
- U302: value STM32L432KCU6 -> STM32L432KCU6TR; DISTPN 497-16578-ND -> 497-STM32L432KCU6TR-ND; MPN STM32L432KCU6 -> STM32L432KCU6TR
- U501: LCSC C46471039 -> (none)
Changed lines of the file:
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@@
 			)
 		)
-		(property "Value" "STM32L432KCU6"
+		(property "Value" "STM32L432KCU6TR"
 			(at 128.27 93.98 0)
 			(show_name no)
@@
 			)
 		)
-		(property "DISTPN" "497-16578-ND"
+		(property "DISTPN" "497-STM32L432KCU6TR-ND"
 			(at 87.63 76.2 0)
 			(hide yes)
@@
 			)
 		)
-		(property "MPN" "STM32L432KCU6"
+		(property "MPN" "STM32L432KCU6TR"
 			(at 0 152.4 0)
 			(hide yes)
@@
 			)
 		)
-		(property "MPN" "GRM033C81E104KE14D"
+		(property "MPN" "GRM033R61A104ME15D"
 			(at 60.96 97.79 0)
 			(hide yes)
@@
 			)
 		)
-		(property "LCSC" "C181047"
+		(property "LCSC" "C408130"
 			(at 60.96 97.79 0)
 			(hide yes)
@@
 			)
 		)
-		(property "MPN" "GRM033C81E104KE14D"
+		(property "MPN" "GRM033R61A104ME15D"
 			(at 68.58 97.79 0)
 			(hide yes)
@@
 			)
 		)
-		(property "LCSC" "C181047"
+		(property "LCSC" "C408130"
 			(at 68.58 97.79 0)
 			(hide yes)
@@
 			)
 		)
-		(property "MPN" "GRM033C81E104KE14D"
+		(property "MPN" "GRM033R61A104ME15D"
 			(at 254 83.82 0)
 			(hide yes)
@@
 			)
 		)
-		(property "LCSC" "C181047"
+		(property "LCSC" "C408130"
 			(at 254 83.82 0)
 			(hide yes)
@@
 		(on_board yes)
 		(in_pos_files no)
-		(dnp no)
+		(dnp yes)
 		(property "Reference" "J301"
 			(at 25.4 180.34 0)
@@
 		(on_board yes)
 		(in_pos_files no)
-		(dnp no)
+		(dnp yes)
 		(property "Reference" "J201"
 			(at 179.07 22.86 0)
@@
 		(on_board yes)
 		(in_pos_files no)
-		(dnp no)
+		(dnp yes)
 		(property "Reference" "J302"
 			(at 33.02 180.34 0)
@@
 		(on_board yes)
 		(in_pos_files no)
-		(dnp no)
+		(dnp yes)
 		(property "Reference" "J303"
 			(at 25.4 186.69 0)
@@
 		(on_board yes)
 		(in_pos_files no)
-		(dnp no)
+		(dnp yes)
 		(property "Reference" "J304"
 			(at 33.02 186.69 0)
@@
 		(on_board yes)
 		(in_pos_files no)
-		(dnp no)
+		(dnp yes)
 		(property "Reference" "J401"
 			(at 218.44 38.1 0)
@@
 			)
 		)
-		(property "LCSC" "C46471039"
-			(at 224.79 76.2 0)
-			(hide yes)
-			(show_name no)
-			(do_not_autoplace no)
-			(effects
-				(font
-					(size 1.524 1.524)
-				)
-			)
-		)
 		(pin "1"
 		)
@@
 			)
 		)
-		(property "MPN" "GRM033C81E104KE14D"
+		(property "MPN" "GRM033R61A104ME15D"
 			(at 179.07 100.33 0)
 			(hide yes)
@@
 			)
 		)
-		(property "LCSC" "C181047"
+		(property "LCSC" "C408130"
 			(at 179.07 100.33 0)
 			(hide yes)
@@
 			)
 		)
-		(property "MPN" "GRM033C81E104KE14D"
+		(property "MPN" "GRM033R61A104ME15D"
 			(at -43.18 262.89 0)
 			(hide yes)
@@
 			)
 		)
-		(property "LCSC" "C181047"
+		(property "LCSC" "C408130"
 			(at 134.62 160.02 0)
 			(hide yes)
@@
 			)
 		)
-		(property "MPN" "GRM033C81E104KE14D"
+		(property "MPN" "GRM033R61A104ME15D"
 			(at 52.07 247.65 0)
 			(hide yes)
@@
 			)
 		)
-		(property "LCSC" "C181047"
+		(property "LCSC" "C408130"
 			(at 229.87 144.78 0)
 			(hide yes)
@@
 			)
 		)
-		(property "MPN" "GRM033C81E104KE14D"
+		(property "MPN" "GRM033R61A104ME15D"
 			(at 43.18 247.65 0)
 			(hide yes)
@@
 			)
 		)
-		(property "LCSC" "C181047"
+		(property "LCSC" "C408130"
 			(at 220.98 144.78 0)
 			(hide yes)
@@
 			)
 		)
-		(property "MPN" "GRM033C81E104KE14D"
+		(property "MPN" "GRM033R61A104ME15D"
 			(at 62.23 72.39 0)
 			(hide yes)
@@
 			)
 		)
-		(property "LCSC" "C181047"
+		(property "LCSC" "C408130"
 			(at 62.23 72.39 0)
 			(hide yes)
@@
 			)
 		)
-		(property "MPN" "GRM033C81E104KE14D"
+		(property "MPN" "GRM033R61A104ME15D"
 			(at -52.07 262.89 0)
 			(hide yes)
@@
 			)
 		)
-		(property "LCSC" "C181047"
+		(property "LCSC" "C408130"
 			(at 125.73 160.02 0)
 			(hide yes)
