File: BoardDesigns/Tags/BitTagv7/BitTagv7.kicad_sch (KiCad schematic)
At the start: 18 parts

Commit message: BitTagv7: upgrade to the KiCad 10 file format, correct the D401 model
Opening and saving the board in KiCad 10 rewrites the pcb, schematic and
project files into the current format, and in passing re-roots nine of the
twelve KISYS3DMOD model paths onto KICAD10_3DMODEL_DIR.

D401's 3D model was wrong: it pointed at a SOT-23 package when the part is a
SOD-923. Now D_SOD-923.step.

Two references remain on KISYS3DMOD -- U405's ADXL362 and Q501's transistor.
Those resolve from a KiCad 5 era location with no KiCad 10 equivalent, so
saving cannot re-root them; they need rewriting by hand.

Note this is a one-way format change: the files no longer open in older KiCad.

Co-Authored-By: Claude Opus 5 <noreply@anthropic.com>
Claude-Session: https://claude.ai/code/session_01QbSYQtdp6pevBXxPYMjfAB
Parts:
- C402, C403, C501, C502, C503: value (none) -> 0.1uf; footprint (none) -> Capacitor_SMD:C_0402_1005Metric
- C404: value (none) -> 4.7uf; footprint (none) -> Capacitor_SMD:C_0402_1005Metric
- D401: value (none) -> D; footprint (none) -> Diode_SMD:D_0402_1005Metric
- J201: value (none) -> CONN_02X04; footprint (none) -> bittag:tagpoints6
- J301, J302, J303, J304: value (none) -> Conn_01x01; footprint (none) -> bittag:taghole1.25mm
- J401: value (none) -> CONN_01X02; footprint (none) -> bittag:MS621
- Q501: value (none) -> Q_NPN_BEC; footprint (none) -> Package_TO_SOT_SMD:SOT-883
- R1: value (none) -> 10k; footprint (none) -> Resistor_SMD:R_0402_1005Metric
- U302: value (none) -> stm32l432; footprint (none) -> Package_DFN_QFN:QFN-32-1EP_5x5mm_P0.5mm_EP3.45x3.45mm
- U405: value (none) -> adxl362; footprint (none) -> bittag:ADXL362
- U501: value (none) -> RV-3028-C7; footprint (none) -> bittag:RV-8803-C7
