File: BoardDesigns/Bases/tagbase-lipo-v1/tagbase-lipo-v1.kicad_pcb (KiCad board)
At the start: 4 copper layers, 50.8 x 69.9 mm, 45 parts, among them J1 Conn_01x04_Female, J101 Conn_02x03_Odd_Even, J102 Conn_02x05_Odd_Even, J104 USB_B_Mini, J5 Conn_01x02, SW1 SW_SPDT, SW2 SW_SPDT, U1 XC6206P332MR, U105 Tactile Switch, U2 XC6808A4C28R-G, U3 AP2112K-1.8, U4 USBLC6-2P6, U5 STM32L432KBU6, U6 TLV9001IDCKR, U7 SN74LVC1T45DCK, U8 SN74LVC1T45DCK

Commit message: tagbase-lipo-v1: test pads, NRST label, and the JLCPCB package
Five 1.5 mm SMD test pads, labelled on silk with references hidden:
J2 '3v3 valid' (PA0 ADC node), J3 'en1.8v', J4 'sck' and J6 'swdio'
(tag side, 1.8 V), all bottom; J7 'Reset' on TAG_RESET, top. All are
excluded from BOM and position files at the symbol, the footprint and
the JLCPCB plugin, so the BOM and CPL are unchanged.

C7 reached NRST through a power:+3V3 symbol relabelled 'NRST', which
read as a +3V3 decoupler. Replaced with a local NRST label; on the
board this is a net rename only.

Regenerated the JLCPCB Gerbers and drills, with the Gerber zip
force-added. Design review updated; all findings closed. Analysis run
2026-10-12_0739 tracked.

Co-Authored-By: Claude Opus 5.5 <noreply@anthropic.com>
Parts:
- added J2: Conn_01x01, TestPoint:TestPoint_Pad_D1.5mm, B.Cu at (133.4, 64.3)
- added J3: Conn_01x01, TestPoint:TestPoint_Pad_D1.5mm, B.Cu at (132.6, 80.2)
- added J4: Conn_01x01, TestPoint:TestPoint_Pad_D1.5mm, B.Cu at (124.6, 86.0)
- added J6: Conn_01x01, TestPoint:TestPoint_Pad_D1.5mm, B.Cu at (117.4, 87.6)
- added J7: Conn_01x01, TestPoint:TestPoint_Pad_D1.5mm, F.Cu at (118.2, 80.4)
Connections:
- net NRST renamed /NRST
Routing:
- net /en1.8v: track 13.8 -> 18.8 mm
- net TAG_RESET: track 22.6 -> 26.8 mm, vias 1 -> 3
- net TAG_SWDIO: track 25.8 -> 29.5 mm
- net /TAG_3V3_Valid: track 5.45 -> 8.45 mm, vias 0 -> 1
- net TAG_SCK: track 18.3 -> 20.7 mm
Other:
- board text added: "3v3 valid"
- board text added: "Reset"
- board text added: "en1.8v"
- board text added: "sck"
- board text added: "swdio"

Commit message: tagbase-lipo-v1: U2 to XC6808ANC28R-G, R2 not fitted
XC6808A4C28R-G (C3682502) is out of stock at LCSC. The only other
standard 4.20 V XC6808 in USP-6B07 is XC6808ANC28R-G (C7123934); it
differs only in the temperature-monitor field. On the xN, pin 5 is NF
and must be left open, so R2 (10k, pin 5 to GND) is now not fitted at
the symbol, the footprint and the JLCPCB plugin. Its footprint stays,
so the A4 can be restored.

The board change is fields only; the Gerbers are content-identical.
The BOM and CPL drop R2 and relabel U2. Review and .kicad-happy.json
updated; analysis run 2026-10-12_0807 replaces 0739.

Co-Authored-By: Claude Opus 5.5 <noreply@anthropic.com>
Parts:
- U2: value XC6808A4C28R-G -> XC6808ANC28R-G
Changed lines of the file:
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@@
 			)
 		)
-		(property "Value" "XC6808A4C28R-G"
+		(property "Value" "XC6808ANC28R-G"
 			(at 0 0 0)
 			(unlocked yes)
@@
 			)
 		)
-		(property "Datasheet" "XC6808A4C28R-G"
+		(property "Datasheet" "XC6808ANC28R-G"
 			(at 0 0 0)
 			(unlocked yes)
@@
 			)
 		)
-		(property "LCSC" "C3682502"
+		(property "LCSC" "C7123934"
 			(at 0 0 0)
 			(unlocked yes)
@@
 			)
 		)
-		(property "MPN" "XC6808A4C28R-G"
+		(property "MPN" "XC6808ANC28R-G"
 			(at 0 0 0)
 			(unlocked yes)
@@
 			)
 		)
-		(attr smd)
+		(attr smd exclude_from_pos_files exclude_from_bom dnp)
 		(duplicate_pad_numbers_are_jumpers no)
 		(fp_line
