File: BoardDesigns/Bases/tagbase-lipo-v1/tagbase-lipo-v1.kicad_sch (KiCad schematic)
At the start: 45 parts, among them J1 Conn_01x04_Female, J101 Conn_02x03_Odd_Even, J102 Conn_02x05_Odd_Even, J104 USB_B_Mini, J5 Conn_01x02, SW1 SW_SPDT, SW2 SW_SPDT, U1 XC6206P332MR, U105 Tactile Switch, U2 XC6808A4C28R-G, U3 AP2112K-1.8, U4 USBLC6-2P6, U5 STM32L432KBU6, U6 TLV9001IDCKR, U7 SN74LVC1T45DCK, U8 SN74LVC1T45DCK

Commit message: tagbase-lipo-v1: test pads, NRST label, and the JLCPCB package
Five 1.5 mm SMD test pads, labelled on silk with references hidden:
J2 '3v3 valid' (PA0 ADC node), J3 'en1.8v', J4 'sck' and J6 'swdio'
(tag side, 1.8 V), all bottom; J7 'Reset' on TAG_RESET, top. All are
excluded from BOM and position files at the symbol, the footprint and
the JLCPCB plugin, so the BOM and CPL are unchanged.

C7 reached NRST through a power:+3V3 symbol relabelled 'NRST', which
read as a +3V3 decoupler. Replaced with a local NRST label; on the
board this is a net rename only.

Regenerated the JLCPCB Gerbers and drills, with the Gerber zip
force-added. Design review updated; all findings closed. Analysis run
2026-10-12_0739 tracked.

Co-Authored-By: Claude Opus 5.5 <noreply@anthropic.com>
Parts:
- added J2, J3, J4, J6, J7: Conn_01x01, TestPoint:TestPoint_Pad_D1.5mm, symbol Connector_Generic:Conn_01x01
Connections:
- net TAG_3V3_Valid: now also J2.1 (Pin_1)
- net TAG_RESET: now also J7.1 (Pin_1)
- net TAG_SCK: now also J4.1 (Pin_1)
- net TAG_SWDIO: now also J6.1 (Pin_1)
- net en1.8v: now also J3.1 (Pin_1)

Commit message: tagbase-lipo-v1: U2 to XC6808ANC28R-G, R2 not fitted
XC6808A4C28R-G (C3682502) is out of stock at LCSC. The only other
standard 4.20 V XC6808 in USP-6B07 is XC6808ANC28R-G (C7123934); it
differs only in the temperature-monitor field. On the xN, pin 5 is NF
and must be left open, so R2 (10k, pin 5 to GND) is now not fitted at
the symbol, the footprint and the JLCPCB plugin. Its footprint stays,
so the A4 can be restored.

The board change is fields only; the Gerbers are content-identical.
The BOM and CPL drop R2 and relabel U2. Review and .kicad-happy.json
updated; analysis run 2026-10-12_0807 replaces 0739.

Co-Authored-By: Claude Opus 5.5 <noreply@anthropic.com>
Parts:
- R2: now not fitted; now left out of the parts list
- U2: value XC6808A4C28R-G -> XC6808ANC28R-G; LCSC C3682502 -> C7123934; MPN XC6808A4C28R-G -> XC6808ANC28R-G
Changed lines of the file:
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@@
 			)
 		)
-		(property "Value" "XC6808A4C28R-G"
+		(property "Value" "XC6808ANC28R-G"
 			(at 58.42 115.57 0)
 			(show_name no)
@@
 			)
 		)
-		(property "Datasheet" "XC6808A4C28R-G"
+		(property "Datasheet" "XC6808ANC28R-G"
 			(at 81.28 123.19 0)
 			(hide yes)
@@
 			)
 		)
-		(property "LCSC" "C3682502"
+		(property "LCSC" "C7123934"
 			(at 81.28 123.19 0)
 			(hide yes)
@@
 			)
 		)
-		(property "MPN" "XC6808A4C28R-G"
+		(property "MPN" "XC6808ANC28R-G"
 			(at 81.28 123.19 0)
 			(hide yes)
@@
 		(body_style 1)
 		(exclude_from_sim no)
-		(in_bom yes)
+		(in_bom no)
 		(on_board yes)
-		(in_pos_files yes)
-		(dnp no)
+		(in_pos_files no)
+		(dnp yes)
 		(property "Reference" "R2"
 			(at 14.732 135.89 0)

Commit message: tagbase-lipo-v1: U4 to TECH PUBLIC, and fix six CPL rotations at source
U4: ST USBLC6-2P6 (C15999) was down to 5 in stock. TECH PUBLIC's
USBLC6-2P6 (C2827693) is a drop-in: same SOT-666 package and identical
pin map in both datasheets. VRWM is 5.0 V vs 5.25 V, but breakdown is
>= 6 V on both. LCSC/MFN changed on the schematic, PCB and plugin DB.
Datasheet added to the shared store.

Rotations: the plugin's community rules were wrong for U1, U3 (SOT-23)
and U6 (SOT-353), and missing for U2, U4 and J104, so these had been
fixed by hand in the JLCPCB preview. jlcpcb/project.db now carries its
own correction table: the 61 community rules plus six reference rules,
mirrored in .kicad-happy.json under fabrication.rotation_corrections.
The CPL differs from the previous commit in exactly those six rows, and
all six were confirmed in the JLCPCB preview.

The Gerbers are content-identical to the previous commit. Render and
schematic PDF regenerated; check_renders.py passes.

Co-Authored-By: Claude Opus 5.5 <noreply@anthropic.com>
Parts:
- U4: LCSC C15999 -> C2827693; MFN STMicroelectronics -> TECH PUBLIC
Changed lines of the file:
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@@
 			)
 		)
-		(property "MFN" "STMicroelectronics"
+		(property "MFN" "TECH PUBLIC"
 			(at 175.26 158.75 0)
 			(hide yes)
@@
 			)
 		)
-		(property "LCSC" "C15999"
+		(property "LCSC" "C2827693"
 			(at 175.26 158.75 0)
 			(hide yes)
