File: BoardDesigns/Tags/UIUCTag/UIUCTag.kicad_sch (KiCad schematic)
At the start: 27 parts, among them J201 CONN_02X04, J301 Conn_01x01, J302 Conn_01x01, J303 Conn_01x01, J304 Conn_01x01, J401 CONN_01X02, Q501 PMBT2222AMBYL, U1 724-AT25FF321A-UUN-T, U2 adxl362, U3 BMP585, U302 STM32L432KCU6TR, U501 RV-3028-C8-32.768kHz-1PPM-TA-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

Commit message: UIUCTag: add U501's LCSC number to the schematic
C46471039 was on the PCB footprint (and so in the production BOM) but
missing from the schematic symbol, so a schematic-driven BOM omitted it
and an Update-PCB field sync could have cleared it. ERC 0, DRC 0 with
schematic parity.

Co-Authored-By: Claude Opus 5.5 <noreply@anthropic.com>
Parts:
- U501: LCSC (none) -> C46471039
Changed lines of the file:
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@@
+			)
+		)
+		(property "LCSC" "C46471039"
+			(at 166.37 231.14 0)
+			(hide yes)
+			(show_name no)
+			(do_not_autoplace no)
+			(effects
+				(font
+					(size 1.27 1.27)
+				)
 			)
 		)
